File: pololu.kicad_sch (KiCad schematic)
At the start: 11 parts, among them J17 pololu, J20 pololu, J21 pololu, J22 pololu, J24 pololu, J25 pololu

Commit message: Fix KiCad 10 footprint library: register kiC library, fix schematic references
Changed lines of the file:
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@@
 		(dnp no)
 		(fields_autoplaced yes)
+		(property "Footprint" "kiC:PinHeader_1x06_P2.54mm_Vertical"
+			(at 86.36 46.99 0)
+			(show_name no)
+			(do_not_autoplace no)
+			(effects
+				(font
+					(size 1.27 1.27)
+				)
+			)
+		)
 		(property "Reference" "J17"
 			(at 86.995 36.83 0)

Commit message: Fix Y1/J17 footprints, update PCB and schematics
Changed lines of the file:
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@@
+		)
+	)
+	(hierarchical_label "reset"
+		(shape input)
+		(at 39.37 74.93 180)
+		(effects
+			(font
+				(size 1.27 1.27)
+			)
+			(justify right)
+		)
+	)
+	(hierarchical_label "enable"
+		(shape input)
+		(at 38.1 80.01 180)
+		(effects
+			(font
+				(size 1.27 1.27)
+			)
+			(justify right)
+		)
+	)
+	(hierarchical_label "sleep"
+		(shape input)
+		(at 38.1 77.47 180)
+		(effects
+			(font
+				(size 1.27 1.27)
+			)
+			(justify right)
 		)
 	)
@@
 		(dnp no)
 		(fields_autoplaced yes)
-		(property "Footprint" "kiC:PinHeader_1x06_P2.54mm_Vertical"
-			(at 86.36 46.99 0)
-			(show_name no)
-			(do_not_autoplace no)
-			(effects
-				(font
-					(size 1.27 1.27)
-				)
-			)
-		)
 		(property "Reference" "J17"
 			(at 86.995 36.83 0)
