File: pololu.kicad_sch (KiCad schematic)
At the start: 11 parts, among them J17 pololu, J20 pololu, J21 pololu, J22 pololu, J24 pololu, J25 pololu

Commit message: Clear remaining KiCad 10-only footprints: SW_Push, kiC, MODULE_MRF24J40MA
Parts:
- J20, J21, J22, J24, J25: footprint kiC:PinHeader_1x06_P2.54mm_Vertical -> (none)
Changed lines of the file:
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@@
 			)
 		)
-		(property "Footprint" "kiC:PinHeader_1x06_P2.54mm_Vertical"
+		(property "Footprint" ""
 			(at 245.11 87.63 0)
 			(hide yes)
@@
 			)
 		)
-		(property "Footprint" "kiC:PinHeader_1x06_P2.54mm_Vertical"
+		(property "Footprint" ""
 			(at 96.52 87.63 0)
 			(hide yes)
@@
 			)
 		)
-		(property "Footprint" "kiC:PinHeader_1x06_P2.54mm_Vertical"
+		(property "Footprint" ""
 			(at 210.82 87.63 0)
 			(hide yes)
@@
 			)
 		)
-		(property "Footprint" "kiC:PinHeader_1x06_P2.54mm_Vertical"
+		(property "Footprint" ""
 			(at 137.16 87.63 0)
 			(hide yes)
@@
 			)
 		)
-		(property "Footprint" "kiC:PinHeader_1x06_P2.54mm_Vertical"
+		(property "Footprint" ""
 			(at 171.45 87.63 0)
 			(hide yes)

Commit message: Extraer footprints de example.kicad_pcb y asignarlos a los esquematicos
Parts:
- J20, J21, J22, J24, J25: footprint (none) -> Connector_PinHeader_2.54mm:PinHeader_1x06_P2.54mm_Vertical
Changed lines of the file:
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@@
 			)
 		)
-		(property "Footprint" ""
+		(property "Footprint" "Connector_PinHeader_2.54mm:PinHeader_1x06_P2.54mm_Vertical"
 			(at 245.11 87.63 0)
 			(hide yes)
@@
 			)
 		)
-		(property "Footprint" ""
+		(property "Footprint" "Connector_PinHeader_2.54mm:PinHeader_1x06_P2.54mm_Vertical"
 			(at 96.52 87.63 0)
 			(hide yes)
@@
 			)
 		)
-		(property "Footprint" ""
+		(property "Footprint" "Connector_PinHeader_2.54mm:PinHeader_1x06_P2.54mm_Vertical"
 			(at 210.82 87.63 0)
 			(hide yes)
@@
 			)
 		)
-		(property "Footprint" ""
+		(property "Footprint" "Connector_PinHeader_2.54mm:PinHeader_1x06_P2.54mm_Vertical"
 			(at 137.16 87.63 0)
 			(hide yes)
@@
 			)
 		)
-		(property "Footprint" ""
+		(property "Footprint" "Connector_PinHeader_2.54mm:PinHeader_1x06_P2.54mm_Vertical"
 			(at 171.45 87.63 0)
 			(hide yes)

Commit message: CNC Raspberry update
Parts:
- added A10, A6, A7, A8, A9: Pololu_Breakout_DRV8825, kiC:HTSSOP-28-EP_IC_TPS61196PWPRQ1, symbol Driver_Motor:Pololu_Breakout_DRV8825
- added JP10, JP13, JP16, JP19, JP22: MS2, Jumper:SolderJumper-2_P1.3mm_Open_RoundedPad1.0x1.5mm, symbol Jumper:Jumper_2_Bridged
- added JP11, JP14, JP17, JP20, JP23, JP25, JP26, JP27, JP28, JP29, JP30, JP31, JP32, JP33, JP34, JP35, JP36, JP37, JP38, JP39, JP40, JP41, JP42, JP43, JP44: MS3, Jumper:SolderJumper-2_P1.3mm_Open_RoundedPad1.0x1.5mm, symbol Jumper:Jumper_2_Bridged
- added JP12, JP15, JP18, JP21, JP9: MS1, Jumper:SolderJumper-2_P1.3mm_Open_RoundedPad1.0x1.5mm, symbol Jumper:Jumper_2_Bridged
- A1, A2, A3, A4, A5: now left out of the parts list
- J15: renamed from J25; footprint Connector_PinHeader_2.54mm:PinHeader_1x06_P2.54mm_Vertical -> Connector_PinHeader_2.54mm:PinHeader_1x04_P2.54mm_Vertical; now left out of the parts list
- J16: renamed from J17; footprint (none) -> Library:PinHeader_1x06_P2.54mm_Vertical; now left out of the parts list
- J17: renamed from J20; footprint Connector_PinHeader_2.54mm:PinHeader_1x06_P2.54mm_Vertical -> Connector_PinHeader_2.54mm:PinHeader_1x04_P2.54mm_Vertical; now left out of the parts list
- J18: renamed from J24; footprint Connector_PinHeader_2.54mm:PinHeader_1x06_P2.54mm_Vertical -> Connector_PinHeader_2.54mm:PinHeader_1x04_P2.54mm_Vertical; now left out of the parts list
- J19: renamed from J22; footprint Connector_PinHeader_2.54mm:PinHeader_1x06_P2.54mm_Vertical -> Connector_PinHeader_2.54mm:PinHeader_1x04_P2.54mm_Vertical; now left out of the parts list
- J20: renamed from J21; footprint Connector_PinHeader_2.54mm:PinHeader_1x06_P2.54mm_Vertical -> Connector_PinHeader_2.54mm:PinHeader_1x04_P2.54mm_Vertical; now left out of the parts list
Connections:
- net +3.3V: now also A1.2 (VDD), A2.2 (VDD), A3.2 (VDD), A4.2 (VDD), A5.2 (VDD); no longer A1.8 (VMOT), A2.8 (VMOT), A3.8 (VMOT), A4.8 (VMOT), A5.8 (VMOT), J16.2 (Pin_2)
- net GND: now also A3.7 (GND), A10.1 (GND), A10.7 (GND), A6.1 (GND), A6.7 (GND), A7.1 (GND), A7.7 (GND), A8.1 (GND), A8.7 (GND), A9.1 (GND), A9.7 (GND)
- net 2B_5: now reaches A5.6 (2B), J20.1 (Pin_1)
- net 2B_5: now also JP40.2 (B)
- net 2A_5: now reaches A5.5 (2A), J20.2 (Pin_2)
- net 2A_5: now also JP39.2 (B)
- net 1A_5: now reaches A5.4 (1A), J20.3 (Pin_3)
- net 1A_5: now also JP38.2 (B)
- net 1B_5: now reaches A5.3 (1B), J20.4 (Pin_4)
- net 1B_5: now also JP37.2 (B)
- net MS1_DRV8825_3: now reaches A3.10 (MS1)
- net MS1_DRV8825_3: now also A8.10 (M0), JP12.2 (B)
- net MS2_DRV8825_3: now reaches A3.11 (MS2)
- net MS2_DRV8825_3: now also A8.11 (M1), JP13.2 (B)
- net MS3_DRV8825_3: now reaches A3.12 (MS3)
- net MS3_DRV8825_3: now also A8.12 (M2), JP14.2 (B)
- net reset: now reaches A3.13 (~{RESET})
- net reset: now also A1.13 (~{RESET}), A2.13 (~{RESET}), A4.13 (~{RESET}), A5.13 (~{RESET}), A10.13 (~{RST}), A6.13 (~{RST}), A7.13 (~{RST}), A8.13 (~{RST}), A9.13 (~{RST})
- net sleep: now reaches A3.14 (~{SLEEP})
- net sleep: now also A1.14 (~{SLEEP}), A2.14 (~{SLEEP}), A4.14 (~{SLEEP}), A5.14 (~{SLEEP}), A10.14 (~{SLP}), A6.14 (~{SLP}), A7.14 (~{SLP}), A8.14 (~{SLP}), A9.14 (~{SLP})
- net step_3: now reaches A3.15 (STEP)
- net step_3: now also A8.15 (STEP)
- net dir_3: now reaches A3.16 (DIR)
- net dir_3: now also A8.16 (DIR)
- net 1B_3: now reaches A3.3 (1B), J18.4 (Pin_4)
- net 1B_3: now also JP41.2 (B)
- net 1A_3: now reaches A3.4 (1A), J18.3 (Pin_3)
- net 1A_3: now also JP42.2 (B)
- net 2A_3: now reaches A3.5 (2A), J18.2 (Pin_2)
- net 2A_3: now also JP43.2 (B)
- net 2B_3: now reaches A3.6 (2B), J18.1 (Pin_1)
- net 2B_3: now also JP44.2 (B)
- net enable_3: now reaches A3.9 (~{ENABLE})
- net enable_3: now also A8.9 (~{EN})
- net MS1_DRV8825_5: now reaches A5.10 (MS1)
- net MS1_DRV8825_5: now also A9.10 (M0), JP21.2 (B)
- net MS2_DRV8825_5: now reaches A5.11 (MS2)
- net MS2_DRV8825_5: now also A9.11 (M1), JP22.2 (B)
- net MS3_DRV8825_5: now reaches A5.12 (MS3)
- net MS3_DRV8825_5: now also A9.12 (M2), JP23.2 (B)
- net step_5: now reaches A5.15 (STEP)
- net step_5: now also A9.15 (STEP)
- net dir_5: now reaches A5.16 (DIR)
- net dir_5: now also A9.16 (DIR)
- net enable_5: now reaches A5.9 (~{ENABLE})
- net enable_5: now also A9.9 (~{EN})
- net 2B_1: now reaches A1.6 (2B), J15.1 (Pin_1)
- net 2B_1: now also JP28.2 (B)
- net 2A_1: now reaches A1.5 (2A), J15.2 (Pin_2)
- net 2A_1: now also JP27.2 (B)
- net 1A_1: now reaches A1.4 (1A), J15.3 (Pin_3)
- net 1A_1: now also JP26.2 (B)
- net 1B_1: now reaches A1.3 (1B), J15.4 (Pin_4)
- net 1B_1: now also JP25.2 (B)
- net MS1_DRV8825_4: now reaches A4.10 (MS1)
- net MS1_DRV8825_4: now also A10.10 (M0), JP18.2 (B)
- net MS2_DRV8825_4: now reaches A4.11 (MS2)
- net MS2_DRV8825_4: now also A10.11 (M1), JP19.2 (B)
- net MS3_DRV8825_4: now reaches A4.12 (MS3)
- net MS3_DRV8825_4: now also A10.12 (M2), JP20.2 (B)
- net step_4: now reaches A4.15 (STEP)
- net step_4: now also A10.15 (STEP)
- net dir_4: now reaches A4.16 (DIR)
- net dir_4: now also A10.16 (DIR)
- net 1B_4: now reaches A4.3 (1B), J19.4 (Pin_4)
- net 1B_4: now also JP33.2 (B)
- net 1A_4: now reaches A4.4 (1A), J19.3 (Pin_3)
- net 1A_4: now also JP34.2 (B)
- net 2A_4: now reaches A4.5 (2A), J19.2 (Pin_2)
- net 2A_4: now also JP35.2 (B)
- net 2B_4: now reaches A4.6 (2B), J19.1 (Pin_1)
- net 2B_4: now also JP36.2 (B)
- net enable_4: now reaches A4.9 (~{ENABLE})
- net enable_4: now also A10.9 (~{EN})
- net MS1_DRV8825_2: now reaches A2.10 (MS1)
- net MS1_DRV8825_2: now also A6.10 (M0), JP15.2 (B)
- net MS2_DRV8825_2: now reaches A2.11 (MS2)
- net MS2_DRV8825_2: now also A6.11 (M1), JP16.2 (B)
- net MS3_DRV8825_2: now reaches A2.12 (MS3)
- net MS3_DRV8825_2: now also A6.12 (M2), JP17.2 (B)
- net step_2: now reaches A2.15 (STEP)
- net step_2: now also A6.15 (STEP)
- net dir_2: now reaches A2.16 (DIR)
- net dir_2: now also A6.16 (DIR)
- net 1B_2: now reaches A2.3 (1B), J17.4 (Pin_4)
- net 1B_2: now also JP29.2 (B)
- net 1A_2: now reaches A2.4 (1A), J17.3 (Pin_3)
- net 1A_2: now also JP30.2 (B)
- net 2A_2: now reaches A2.5 (2A), J17.2 (Pin_2)
- net 2A_2: now also JP31.2 (B)
- net 2B_2: now reaches A2.6 (2B), J17.1 (Pin_1)
- net 2B_2: now also JP32.2 (B)
- net enable_2: now reaches A2.9 (~{ENABLE})
- net enable_2: now also A6.9 (~{EN})
- net MS1: now reaches J16.3 (Pin_3)
- net MS1: now also JP12.1 (A), JP15.1 (A), JP18.1 (A), JP21.1 (A), JP9.1 (A)
- net MS2: now reaches J16.4 (Pin_4)
- net MS2: now also JP10.1 (A), JP13.1 (A), JP16.1 (A), JP19.1 (A), JP22.1 (A)
- net MS3: now reaches J16.5 (Pin_5)
- net MS3: now also JP11.1 (A), JP14.1 (A), JP17.1 (A), JP20.1 (A), JP23.1 (A)
- net MS1_DRV8825_1: now reaches A1.10 (MS1)
- net MS1_DRV8825_1: now also A7.10 (M0), JP9.2 (B)
- net MS2_DRV8825_1: now reaches A1.11 (MS2)
- net MS2_DRV8825_1: now also A7.11 (M1), JP10.2 (B)
- net MS3_DRV8825_1: now reaches A1.12 (MS3)
- net MS3_DRV8825_1: now also A7.12 (M2), JP11.2 (B)
- net step_1: now reaches A1.15 (STEP)
- net step_1: now also A7.15 (STEP)
- net dir_1: now reaches A1.16 (DIR)
- net dir_1: now also A7.16 (DIR)
- net enable_1: now reaches A1.9 (~{ENABLE})
- net enable_1: now also A7.9 (~{EN})
- removed net +5V: A1.2 (VDD), A2.2 (VDD), A3.2 (VDD), A4.2 (VDD), A5.2 (VDD), J16.1 (Pin_1)
- new net: A6.5 (B1), JP31.1 (A)
- new net: A8.4 (A1), JP41.1 (A)
- new net: A6.4 (A1), JP29.1 (A)
- new net: A10.3 (A2), JP34.1 (A)
- new net: A6.6 (B2), JP32.1 (A)
- new net: A10.4 (A1), JP33.1 (A)
- new net: A10.5 (B1), JP35.1 (A)
- new net: A9.3 (A2), JP38.1 (A)
- new net: A9.4 (A1), JP37.1 (A)
- new net: A9.5 (B1), JP39.1 (A)
- new net: A9.6 (B2), JP40.1 (A)
- new net: A7.6 (B2), JP28.1 (A)
- new net: A7.3 (A2), JP26.1 (A)
- new net: A7.4 (A1), JP25.1 (A)
- new net: A7.5 (B1), JP27.1 (A)
- new net: A6.3 (A2), JP30.1 (A)
- new net: A8.6 (B2), JP44.1 (A)
- new net: A10.6 (B2), JP36.1 (A)
- new net: A8.3 (A2), JP42.1 (A)
- new net: A8.5 (B1), JP43.1 (A)
- new net FLT_1: A7.2 (~{FLT})
- new net FLT_2: A6.2 (~{FLT})
- new net FLT_3: A8.2 (~{FLT})
- new net FLT_4: A10.2 (~{FLT})
- new net FLT_5: A9.2 (~{FLT})
- new net VCC: A1.8 (VMOT), A10.8 (VMOT), A2.8 (VMOT), A3.8 (VMOT), A4.8 (VMOT), A5.8 (VMOT), A6.8 (VMOT), A7.8 (VMOT), A8.8 (VMOT), A9.8 (VMOT), J16.1 (Pin_1)
- new net VDD: J16.2 (Pin_2)
- no-connect marks 0 -> 1
Other:
- moved on the sheet: A1, A2, A3, A4, A5, J15, J16, J17, J18, J19, J20
