File: osc_ft232.kicad_sch (KiCad schematic)
At the start: 3 parts, among them Y2 6MHZ

Commit message: feat: PCB layout updates, schematic changes, fp-lib-table config
- cnc_pic32.kicad_pcb: component repositioning, board outline, text formatting
- cnc_pic32.kicad_prl/pro: project settings updates
- fp-lib-table: add Library path to Library.pretty
- mcu.kicad_sch: PIC32 pin configuration updates
- zigbee.kicad_sch: MRF24J40 module updates
- oscilator.kicad_sch: crystal configuration
- power.kicad_sch/power_ft232.kicad_sch: power supply updates
- oled.kicad_sch: OLED display connections
- idc.kicad_sch: IDC connector updates
- osc_ft232.kicad_sch: FT232 crystal
Parts:
- renumbered C16 to C21, C17 to C22
Changed lines of the file:
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@@
 		(in_pos_files yes)
 		(dnp no)
-		(property "Reference" "C17"
+		(property "Reference" "C22"
 			(at 163.83 95.25 0)
 			(show_name no)
@@
 			(project "cnc_pic32"
 				(path "/13dbfc1f-be47-44ca-9042-3d6a9a657d7d/22a12b0c-67ed-4f76-a580-7ac736b63dbd/c46be0f3-d253-4db4-864e-55347475c86f"
-					(reference "C17")
+					(reference "C22")
 					(unit 1)
 				)
@@
 		(in_pos_files yes)
 		(dnp no)
-		(property "Reference" "#PWR019"
+		(property "Reference" "#PWR032"
 			(at 148.59 110.49 0)
 			(hide yes)
@@
 			(project "cnc_pic32"
 				(path "/13dbfc1f-be47-44ca-9042-3d6a9a657d7d/22a12b0c-67ed-4f76-a580-7ac736b63dbd/c46be0f3-d253-4db4-864e-55347475c86f"
-					(reference "#PWR019")
+					(reference "#PWR032")
 					(unit 1)
 				)
@@
 		(in_pos_files yes)
 		(dnp no)
-		(property "Reference" "#PWR020"
+		(property "Reference" "#PWR033"
 			(at 153.67 83.82 0)
 			(hide yes)
@@
 			(project "cnc_pic32"
 				(path "/13dbfc1f-be47-44ca-9042-3d6a9a657d7d/22a12b0c-67ed-4f76-a580-7ac736b63dbd/c46be0f3-d253-4db4-864e-55347475c86f"
-					(reference "#PWR020")
+					(reference "#PWR033")
 					(unit 1)
 				)
@@
 		(in_pos_files yes)
 		(dnp no)
-		(property "Reference" "C16"
+		(property "Reference" "C21"
 			(at 139.7 95.25 0)
 			(show_name no)
@@
 			(project "cnc_pic32"
 				(path "/13dbfc1f-be47-44ca-9042-3d6a9a657d7d/22a12b0c-67ed-4f76-a580-7ac736b63dbd/c46be0f3-d253-4db4-864e-55347475c86f"
-					(reference "C16")
-					(unit 1)
-				)
+					(reference "C21")
+					(unit 1)
+				)
