File: osc_ft232.kicad_sch (KiCad schematic)
At the start: 3 parts, among them Y2 6MHZ

Commit message: CNC Raspberry update
Parts:
- renumbered C16 to C21, C17 to C22
Changed lines of the file:
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@@
 (kicad_sch
-	(version 20220115)
+	(version 20260306)
 	(generator "eeschema")
+	(generator_version "10.0")
 	(paper "A4")
 	(junction
@@
 		(unit 1)
 		(body_style 1)
+		(exclude_from_sim no)
+		(in_bom yes)
+		(on_board yes)
 		(in_pos_files yes)
-		(property "Reference" "C17"
+		(dnp no)
+		(property "Reference" "C22"
 			(at 163.83 95.25 0)
+			(show_name no)
+			(do_not_autoplace no)
 			(effects
 				(font
@@
 		(property "Value" "15p"
 			(at 163.83 97.79 0)
+			(show_name no)
+			(do_not_autoplace no)
 			(effects
 				(font
@@
 			(at 160.9852 100.33 0)
 			(hide yes)
+			(show_name no)
+			(do_not_autoplace no)
 			(effects
 				(font
@@
 			(at 160.02 96.52 0)
 			(hide yes)
+			(show_name no)
+			(do_not_autoplace no)
 			(effects
 				(font
@@
 		(property "Description" ""
 			(at 160.02 96.52 0)
+			(show_name no)
+			(do_not_autoplace no)
 			(effects
 				(font
@@
 			(project "cnc_pic32"
 				(path "/13dbfc1f-be47-44ca-9042-3d6a9a657d7d/22a12b0c-67ed-4f76-a580-7ac736b63dbd/c46be0f3-d253-4db4-864e-55347475c86f"
-					(reference "C17")
+					(reference "C22")
 					(unit 1)
 				)
@@
 		(unit 1)
 		(body_style 1)
+		(exclude_from_sim no)
+		(in_bom yes)
+		(on_board yes)
 		(in_pos_files yes)
-		(property "Reference" "#PWR019"
+		(dnp no)
+		(property "Reference" "#PWR032"
 			(at 148.59 110.49 0)
 			(hide yes)
+			(show_name no)
+			(do_not_autoplace no)
 			(effects
 				(font
@@
 		(property "Value" "GND"
 			(at 148.59 109.22 0)
+			(show_name no)
+			(do_not_autoplace no)
 			(effects
 				(font
@@
 			(at 148.59 104.14 0)
 			(hide yes)
+			(show_name no)
+			(do_not_autoplace no)
 			(effects
 				(font
@@
 			(at 148.59 104.14 0)
 			(hide yes)
+			(show_name no)
+			(do_not_autoplace no)
 			(effects
 				(font
@@
 		(property "Description" ""
 			(at 148.59 104.14 0)
+			(show_name no)
+			(do_not_autoplace no)
 			(effects
 				(font
@@
 			(project "cnc_pic32"
 				(path "/13dbfc1f-be47-44ca-9042-3d6a9a657d7d/22a12b0c-67ed-4f76-a580-7ac736b63dbd/c46be0f3-d253-4db4-864e-55347475c86f"
-					(reference "#PWR019")
+					(reference "#PWR032")
 					(unit 1)
 				)
@@
 		(unit 1)
 		(body_style 1)
+		(exclude_from_sim no)
+		(in_bom yes)
+		(on_board yes)
 		(in_pos_files yes)
-		(property "Reference" "#PWR020"
+		(dnp no)
+		(property "Reference" "#PWR033"
 			(at 153.67 83.82 0)
 			(hide yes)
+			(show_name no)
+			(do_not_autoplace no)
 			(effects
 				(font
@@
 		(property "Value" "GND"
 			(at 153.67 82.55 0)
+			(show_name no)
+			(do_not_autoplace no)
 			(effects
 				(font
@@
 			(at 153.67 77.47 0)
 			(hide yes)
+			(show_name no)
+			(do_not_autoplace no)
 			(effects
 				(font
@@
 			(at 153.67 77.47 0)
 			(hide yes)
+			(show_name no)
+			(do_not_autoplace no)
 			(effects
 				(font
@@
 		(property "Description" ""
 			(at 153.67 77.47 0)
+			(show_name no)
+			(do_not_autoplace no)
 			(effects
 				(font
@@
 			(project "cnc_pic32"
 				(path "/13dbfc1f-be47-44ca-9042-3d6a9a657d7d/22a12b0c-67ed-4f76-a580-7ac736b63dbd/c46be0f3-d253-4db4-864e-55347475c86f"
-					(reference "#PWR020")
+					(reference "#PWR033")
 					(unit 1)
 				)
@@
 		(unit 1)
 		(body_style 1)
+		(exclude_from_sim no)
+		(in_bom yes)
+		(on_board yes)
 		(in_pos_files yes)
-		(property "Reference" "C16"
+		(dnp no)
+		(property "Reference" "C21"
 			(at 139.7 95.25 0)
+			(show_name no)
+			(do_not_autoplace no)
 			(effects
 				(font
@@
 		(property "Value" "15p"
 			(at 139.7 97.79 0)
+			(show_name no)
+			(do_not_autoplace no)
 			(effects
 				(font
@@
 			(at 136.8552 100.33 0)
 			(hide yes)
+			(show_name no)
+			(do_not_autoplace no)
 			(effects
 				(font
@@
 			(at 135.89 96.52 0)
 			(hide yes)
+			(show_name no)
+			(do_not_autoplace no)
 			(effects
 				(font
@@
 		(property "Description" ""
 			(at 135.89 96.52 0)
+			(show_name no)
+			(do_not_autoplace no)
 			(effects
 				(font
@@
 			(project "cnc_pic32"
 				(path "/13dbfc1f-be47-44ca-9042-3d6a9a657d7d/22a12b0c-67ed-4f76-a580-7ac736b63dbd/c46be0f3-d253-4db4-864e-55347475c86f"
-					(reference "C16")
+					(reference "C21")
 					(unit 1)
 				)
@@
 		(unit 1)
 		(body_style 1)
+		(exclude_from_sim no)
+		(in_bom yes)
+		(on_board yes)
 		(in_pos_files yes)
+		(dnp no)
 		(property "Reference" "Y2"
 			(at 160.02 88.5191 0)
+			(show_name no)
+			(do_not_autoplace no)
 			(effects
 				(font
@@
 		(property "Value" "6MHZ"
 			(at 140.462 85.09 0)
+			(show_name no)
+			(do_not_autoplace no)
 			(effects
 				(font
@@
 			(at 148.59 92.71 0)
 			(hide yes)
+			(show_name no)
+			(do_not_autoplace no)
 			(effects
 				(font
@@
 			(at 148.59 92.71 0)
 			(hide yes)
+			(show_name no)
+			(do_not_autoplace no)
 			(effects
 				(font
@@
 		(property "Description" ""
 			(at 148.59 92.71 0)
-			(effects
-				(font
+			(show_name no)
+			(do_not_autoplace no)
+			(effects
+				(font
