File: tp_ft232.kicad_sch (KiCad schematic)
At the start: 10 parts, among them J10 tp_ft232_, J11 tp_ft232_, J12 tp_ft232_, J16 tp_ft232_, J6 tp_ft232_, J7 tp_ft232_, J8 tp_ft232_, J9 tp_ft232_

Commit message: Fix KiCad 10 footprint library: register kiC library, fix schematic references
Parts:
- J10, J11, J12, J6, J7, J8, J9: footprint Connector_Pin:pad_0508 -> kiC:pad_0508
- J16: footprint Connector_Pin:Pin_D1.5mmx1mm -> kiC:Pin_D1.5mmx1mm
Changed lines of the file:
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@@
 			)
 		)
-		(property "Footprint" "Connector_Pin:pad_0508"
+		(property "Footprint" "kiC:pad_0508"
 			(at 123.19 138.43 0)
 			(hide yes)
@@
 			)
 		)
-		(property "Footprint" "Connector_Pin:pad_0508"
+		(property "Footprint" "kiC:pad_0508"
 			(at 118.11 107.95 0)
 			(hide yes)
@@
 			)
 		)
-		(property "Footprint" "Connector_Pin:pad_0508"
+		(property "Footprint" "kiC:pad_0508"
 			(at 118.11 92.71 0)
 			(hide yes)
@@
 			)
 		)
-		(property "Footprint" "Connector_Pin:pad_0508"
+		(property "Footprint" "kiC:pad_0508"
 			(at 118.11 97.79 0)
 			(hide yes)
@@
 			)
 		)
-		(property "Footprint" "Connector_Pin:pad_0508"
+		(property "Footprint" "kiC:pad_0508"
 			(at 124.46 132.08 0)
 			(hide yes)
@@
 			)
 		)
-		(property "Footprint" "Connector_Pin:Pin_D1.5mmx1mm"
+		(property "Footprint" "kiC:Pin_D1.5mmx1mm"
 			(at 203.2 115.57 0)
 			(hide yes)
@@
 			)
 		)
-		(property "Footprint" "Connector_Pin:pad_0508"
+		(property "Footprint" "kiC:pad_0508"
 			(at 118.11 105.41 0)
 			(hide yes)
@@
 			)
 		)
-		(property "Footprint" "Connector_Pin:pad_0508"
+		(property "Footprint" "kiC:pad_0508"
 			(at 118.11 102.87 0)
 			(hide yes)

Commit message: feat: tp_ft232 hierarchical labels + ft232 sheet pins
- Convert 9 local labels in tp_ft232 to hierarchical labels
- Remove conflicting global labels (FT_CTS, FT_RTS)
- Add 9 sheet pins to tp_ft232 box in ft232.kicad_sch
- Restructure cnc-pic32 skill to .opencode/skills/cnc-pic32/SKILL.md
Connections:
- net FT_RTS renamed FT_RST
Changed lines of the file:
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@@
 		)
 	)
-	(label "FT_CTS"
-		(at 128.27 119.38 180)
+	(hierarchical_label "FT_CTS"
+		(shape input)
+		(at 134.62 119.38 0)
 		(effects
 			(font
 				(size 1.27 1.27)
 			)
-			(justify right bottom)
+			(justify left)
 		)
 	)
-	(label "FT_DRS"
+	(hierarchical_label "FT_DRS"
+		(shape input)
 		(at 135.89 102.87 0)
 		(effects
@@
 				(size 1.27 1.27)
 			)
-			(justify left bottom)
+			(justify left)
 		)
 	)
-	(label "FT_TXD_EN"
+	(hierarchical_label "FT_TXD_EN"
+		(shape input)
 		(at 135.89 105.41 0)
 		(effects
@@
 				(size 1.27 1.27)
 			)
-			(justify left bottom)
+			(justify left)
 		)
 	)
-	(label "FT_DCD"
+	(hierarchical_label "FT_DCD"
+		(shape input)
 		(at 135.89 97.79 0)
 		(effects
@@
 				(size 1.27 1.27)
 			)
-			(justify left bottom)
+			(justify left)
 		)
 	)
-	(label "FT_RST"
-		(at 128.27 115.57 180)
+	(hierarchical_label "FT_RST"
+		(shape input)
+		(at 134.62 115.57 0)
 		(effects
 			(font
 				(size 1.27 1.27)
 			)
-			(justify right bottom)
+			(justify left)
 		)
 	)
-	(label "FT_RI"
+	(hierarchical_label "FT_RI"
+		(shape input)
 		(at 135.89 92.71 0)
 		(effects
@@
 				(size 1.27 1.27)
 			)
-			(justify left bottom)
+			(justify left)
 		)
 	)
-	(label "FT_PWR_EN"
+	(hierarchical_label "FT_PWR_EN"
+		(shape input)
 		(at 135.89 107.95 0)
 		(effects
@@
 				(size 1.27 1.27)
 			)
-			(justify left bottom)
+			(justify left)
 		)
 	)
-	(label "FT_RST"
+	(hierarchical_label "FT_RST"
+		(shape input)
 		(at 146.05 138.43 0)
 		(effects
@@
 				(size 1.27 1.27)
 			)
-			(justify left bottom)
+			(justify left)
 		)
 	)
-	(label "FT_DTR"
+	(hierarchical_label "FT_DTR"
+		(shape input)
 		(at 147.32 132.08 0)
 		(effects
@@
 				(size 1.27 1.27)
 			)
-			(justify left bottom)
+			(justify left)
 		)
 	)
@@
 		(property "Intersheetrefs" "${INTERSHEET_REFS}"
 			(at 208.5437 66.04 0)
-			(hide yes)
-			(show_name no)
-			(do_not_autoplace no)
-			(effects
-				(font
-					(size 1.27 1.27)
-				)
-				(justify left)
-			)
-		)
-	)
-	(global_label "FT_CTS"
-		(shape input)
-		(at 134.62 119.38 0)
-		(fields_autoplaced yes)
-		(effects
-			(font
-				(size 1.27 1.27)
-			)
-			(justify left)
-		)
-		(property "Intersheetrefs" "${INTERSHEET_REFS}"
-			(at 143.9967 119.38 0)
 			(hide yes)
 			(show_name no)
@@
 			)
 		)
-	)
-	(global_label "FT_RTS"
-		(shape input)
-		(at 134.62 115.57 0)
-		(fields_autoplaced yes)
-		(effects
-			(font
-				(size 1.27 1.27)
-			)
-			(justify left)
-		)
-		(property "Intersheetrefs" "${INTERSHEET_REFS}"
-			(at 143.9967 115.57 0)
-			(hide yes)
-			(show_name no)
-			(do_not_autoplace no)
-			(effects
-				(font
-					(size 1.27 1.27)
-				)
-				(justify left)
-			)
-		)

Commit message: fix: tp_ft232 footprints kiC:pad_0508 + kiC:Pin_D1.5mmx1mm → Library:connector_pin1
Parts:
- J10, J11, J12, J6, J7, J8, J9: footprint kiC:pad_0508 -> Library:connector_pin1
- J16: footprint kiC:Pin_D1.5mmx1mm -> Library:connector_pin1
Changed lines of the file:
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@@
-		)
-	)
-	(hierarchical_label "FT_CTS"
-		(shape input)
-		(at 134.62 119.38 0)
-		(effects
-			(font
-				(size 1.27 1.27)
-			)
-			(justify left)
-		)
-	)
-	(hierarchical_label "FT_DRS"
-		(shape input)
-		(at 135.89 102.87 0)
-		(effects
-			(font
-				(size 1.27 1.27)
-			)
-			(justify left)
-		)
-	)
-	(hierarchical_label "FT_TXD_EN"
-		(shape input)
-		(at 135.89 105.41 0)
-		(effects
-			(font
-				(size 1.27 1.27)
-			)
-			(justify left)
-		)
-	)
-	(hierarchical_label "FT_DCD"
-		(shape input)
-		(at 135.89 97.79 0)
-		(effects
-			(font
-				(size 1.27 1.27)
-			)
-			(justify left)
-		)
-	)
-	(hierarchical_label "FT_RST"
-		(shape input)
-		(at 134.62 115.57 0)
-		(effects
-			(font
-				(size 1.27 1.27)
-			)
-			(justify left)
-		)
-	)
-	(hierarchical_label "FT_RI"
-		(shape input)
-		(at 135.89 92.71 0)
-		(effects
-			(font
-				(size 1.27 1.27)
-			)
-			(justify left)
-		)
-	)
-	(hierarchical_label "FT_PWR_EN"
-		(shape input)
-		(at 135.89 107.95 0)
-		(effects
-			(font
-				(size 1.27 1.27)
-			)
-			(justify left)
-		)
-	)
-	(hierarchical_label "FT_RST"
-		(shape input)
-		(at 146.05 138.43 0)
-		(effects
-			(font
-				(size 1.27 1.27)
-			)
-			(justify left)
-		)
-	)
-	(hierarchical_label "FT_DTR"
-		(shape input)
-		(at 147.32 132.08 0)
-		(effects
-			(font
-				(size 1.27 1.27)
-			)
-			(justify left)
 		)
 	)
@@
 		)
 	)
+	(hierarchical_label "FT_CTS"
+		(shape input)
+		(at 134.62 119.38 0)
+		(effects
+			(font
+				(size 1.27 1.27)
+			)
+			(justify left)
+		)
+	)
+	(hierarchical_label "FT_DRS"
+		(shape input)
+		(at 135.89 102.87 0)
+		(effects
+			(font
+				(size 1.27 1.27)
+			)
+			(justify left)
+		)
+	)
+	(hierarchical_label "FT_TXD_EN"
+		(shape input)
+		(at 135.89 105.41 0)
+		(effects
+			(font
+				(size 1.27 1.27)
+			)
+			(justify left)
+		)
+	)
+	(hierarchical_label "FT_DCD"
+		(shape input)
+		(at 135.89 97.79 0)
+		(effects
+			(font
+				(size 1.27 1.27)
+			)
+			(justify left)
+		)
+	)
 	(hierarchical_label "TX_MCU"
 		(shape input)
@@
 		)
 	)
+	(hierarchical_label "FT_RST"
+		(shape input)
+		(at 134.62 115.57 0)
+		(effects
+			(font
+				(size 1.27 1.27)
+			)
+			(justify left)
+		)
+	)
+	(hierarchical_label "FT_RI"
+		(shape input)
+		(at 135.89 92.71 0)
+		(effects
+			(font
+				(size 1.27 1.27)
+			)
+			(justify left)
+		)
+	)
+	(hierarchical_label "FT_PWR_EN"
+		(shape input)
+		(at 135.89 107.95 0)
+		(effects
+			(font
+				(size 1.27 1.27)
+			)
+			(justify left)
+		)
+	)
+	(hierarchical_label "FT_RST"
+		(shape input)
+		(at 146.05 138.43 0)
+		(effects
+			(font
+				(size 1.27 1.27)
+			)
+			(justify left)
+		)
+	)
 	(hierarchical_label "RX_MCU"
 		(shape input)
@@
 			)
 			(justify right)
+		)
+	)
+	(hierarchical_label "FT_DTR"
+		(shape input)
+		(at 147.32 132.08 0)
+		(effects
+			(font
+				(size 1.27 1.27)
+			)
+			(justify left)
 		)
 	)
@@
 			)
 		)
-		(property "Footprint" "kiC:pad_0508"
+		(property "Footprint" "Library:connector_pin1"
 			(at 123.19 138.43 0)
 			(hide yes)
@@
 			)
 		)
-		(property "Footprint" "kiC:pad_0508"
+		(property "Footprint" "Library:connector_pin1"
 			(at 118.11 107.95 0)
 			(hide yes)
@@
 			)
 		)
-		(property "Footprint" "kiC:pad_0508"
+		(property "Footprint" "Library:connector_pin1"
 			(at 118.11 92.71 0)
 			(hide yes)
@@
 			)
 		)
-		(property "Footprint" "kiC:pad_0508"
+		(property "Footprint" "Library:connector_pin1"
 			(at 118.11 97.79 0)
 			(hide yes)
@@
 			)
 		)
-		(property "Footprint" "kiC:pad_0508"
+		(property "Footprint" "Library:connector_pin1"
 			(at 124.46 132.08 0)
 			(hide yes)
@@
 			)
 		)
-		(property "Footprint" "kiC:Pin_D1.5mmx1mm"
+		(property "Footprint" "Library:connector_pin1"
 			(at 203.2 115.57 0)
 			(hide yes)
@@
 			)
 		)
-		(property "Footprint" "kiC:pad_0508"
+		(property "Footprint" "Library:connector_pin1"
 			(at 118.11 105.41 0)
 			(hide yes)
@@
 			)
 		)
-		(property "Footprint" "kiC:pad_0508"
+		(property "Footprint" "Library:connector_pin1"
 			(at 118.11 102.87 0)
 			(hide yes)

Commit message: feat: 25 hierarchical labels for 5 Pololus + fix J4/J15/J17/TP17 footprints + USB pin6→SH
- pololu.kicad_sch: 5→25 hierarchical labels (reset_N, sleep_N, enable_N, step_N, dir_N) with wires to each Pololu A4988
- pololu.kicad_sch: J17 footprint kiC:PinHeader → Library:PinHeader_1x06_P2.54mm_Vertical
- cnc_pic32.kicad_sch: expanded Pololu sheet box with 25 named sheet pins
- buttons.kicad_sch: all SW switches → Button_Switch_SMD:SW_SPST_CK_RS282G05A3
- tp_ft232.kicad_sch: kiC:pad_0508 + kiC:Pin_D1.5mmx1mm → Library:connector_pin1
- usb_conector_Ft232.kicad_sch: J4/J15 kiC:Pin_D1.5mmx1mm → Library:connector_pin1, J5 pin 6→SH
- Usb_pic32.kicad_sch: TP17 kiC:Pin_D1.5mmx1mm → Library:connector_pin1, J18 pin 6→SH
Parts:
- renumbered J9 to J10, J10 to J11, J11 to J12, J12 to J13, J16 to J14, J6 to J7, J7 to J8, J8 to J9, JP2 to JP1, JP1 to JP2
Changed lines of the file:
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@@
 		(in_pos_files yes)
 		(dnp no)
-		(property "Reference" "J11"
+		(property "Reference" "J12"
 			(at 121.92 137.16 0)
 			(show_name no)
@@
 			(project "cnc_pic32"
 				(path "/13dbfc1f-be47-44ca-9042-3d6a9a657d7d/22a12b0c-67ed-4f76-a580-7ac736b63dbd/aa6b2b7f-e067-4903-af41-a51929953e3c"
-					(reference "J11")
+					(reference "J12")
 					(unit 1)
 				)
@@
 		(in_pos_files yes)
 		(dnp no)
-		(property "Reference" "J10"
+		(property "Reference" "J11"
 			(at 116.84 106.68 0)
 			(show_name no)
@@
 			(project "cnc_pic32"
 				(path "/13dbfc1f-be47-44ca-9042-3d6a9a657d7d/22a12b0c-67ed-4f76-a580-7ac736b63dbd/aa6b2b7f-e067-4903-af41-a51929953e3c"
-					(reference "J10")
+					(reference "J11")
 					(unit 1)
 				)
@@
 		(in_pos_files yes)
 		(dnp no)
-		(property "Reference" "J6"
+		(property "Reference" "J7"
 			(at 116.84 91.44 0)
 			(show_name no)
@@
 			(project "cnc_pic32"
 				(path "/13dbfc1f-be47-44ca-9042-3d6a9a657d7d/22a12b0c-67ed-4f76-a580-7ac736b63dbd/aa6b2b7f-e067-4903-af41-a51929953e3c"
-					(reference "J6")
+					(reference "J7")
 					(unit 1)
 				)
@@
 		(in_pos_files yes)
 		(dnp no)
-		(property "Reference" "J7"
+		(property "Reference" "J8"
 			(at 116.84 96.52 0)
 			(show_name no)
@@
 			(project "cnc_pic32"
 				(path "/13dbfc1f-be47-44ca-9042-3d6a9a657d7d/22a12b0c-67ed-4f76-a580-7ac736b63dbd/aa6b2b7f-e067-4903-af41-a51929953e3c"
-					(reference "J7")
+					(reference "J8")
 					(unit 1)
 				)
@@
 		(in_pos_files yes)
 		(dnp no)
-		(property "Reference" "J12"
+		(property "Reference" "J13"
 			(at 123.19 130.81 0)
 			(show_name no)
@@
 			(project "cnc_pic32"
 				(path "/13dbfc1f-be47-44ca-9042-3d6a9a657d7d/22a12b0c-67ed-4f76-a580-7ac736b63dbd/aa6b2b7f-e067-4903-af41-a51929953e3c"
-					(reference "J12")
+					(reference "J13")
 					(unit 1)
 				)
@@
 		(dnp no)
 		(fields_autoplaced yes)
-		(property "Reference" "JP2"
+		(property "Reference" "JP1"
 			(at 135.89 59.69 0)
 			(show_name no)
@@
 			(project "cnc_pic32"
 				(path "/13dbfc1f-be47-44ca-9042-3d6a9a657d7d/22a12b0c-67ed-4f76-a580-7ac736b63dbd/aa6b2b7f-e067-4903-af41-a51929953e3c"
-					(reference "JP2")
+					(reference "JP1")
 					(unit 1)
 				)
@@
 		(in_pos_files yes)
 		(dnp no)
-		(property "Reference" "J16"
+		(property "Reference" "J14"
 			(at 201.93 114.3 0)
 			(show_name no)
@@
 			(project "cnc_pic32"
 				(path "/13dbfc1f-be47-44ca-9042-3d6a9a657d7d/22a12b0c-67ed-4f76-a580-7ac736b63dbd/aa6b2b7f-e067-4903-af41-a51929953e3c"
-					(reference "J16")
+					(reference "J14")
 					(unit 1)
 				)
@@
 		(in_pos_files yes)
 		(dnp no)
-		(property "Reference" "J9"
+		(property "Reference" "J10"
 			(at 116.84 104.14 0)
 			(show_name no)
@@
 			(project "cnc_pic32"
 				(path "/13dbfc1f-be47-44ca-9042-3d6a9a657d7d/22a12b0c-67ed-4f76-a580-7ac736b63dbd/aa6b2b7f-e067-4903-af41-a51929953e3c"
-					(reference "J9")
+					(reference "J10")
 					(unit 1)
 				)
@@
 		(dnp no)
 		(fields_autoplaced yes)
-		(property "Reference" "JP1"
+		(property "Reference" "JP2"
 			(at 187.96 59.69 0)
 			(show_name no)
@@
 			(project "cnc_pic32"
 				(path "/13dbfc1f-be47-44ca-9042-3d6a9a657d7d/22a12b0c-67ed-4f76-a580-7ac736b63dbd/aa6b2b7f-e067-4903-af41-a51929953e3c"
-					(reference "JP1")
+					(reference "JP2")
 					(unit 1)
 				)
@@
 		(in_pos_files yes)
 		(dnp no)
-		(property "Reference" "J8"
+		(property "Reference" "J9"
 			(at 116.84 101.6 0)
 			(show_name no)
@@
 			(project "cnc_pic32"
 				(path "/13dbfc1f-be47-44ca-9042-3d6a9a657d7d/22a12b0c-67ed-4f76-a580-7ac736b63dbd/aa6b2b7f-e067-4903-af41-a51929953e3c"
-					(reference "J8")
-					(unit 1)
-				)
+					(reference "J9")
+					(unit 1)
+				)

Commit message: feat: PCB layout updates, schematic changes, remove freerouting.dsn
Changed lines of the file:
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@@
-	(wire
-		(pts
-			(xy 128.27 115.57) (xy 134.62 115.57)
-		)
-		(stroke
-			(width 0)
-			(type default)
-		)
-	)
 	(wire
 		(pts
@@
 	(wire
 		(pts
-			(xy 128.27 119.38) (xy 134.62 119.38)
-		)
-		(stroke
-			(width 0)
-			(type default)
-		)
-	)
-	(wire
-		(pts
 			(xy 187.96 77.47) (xy 187.96 69.85)
 		)
@@
 		)
 	)
+	(label "FT_TXD_EN"
+		(at 15.9235 7.1757 180)
+		(effects
+			(font
+				(size 1.27 1.27)
+			)
+			(justify right bottom)
+		)
+	)
+	(label "FT_TXD_EN"
+		(at 21.0035 12.2557 180)
+		(effects
+			(font
+				(size 1.27 1.27)
+			)
+			(justify right bottom)
+		)
+	)
+	(label "FT_RESET"
+		(at 66.7235 12.2557 0)
+		(effects
+			(font
+				(size 1.27 1.27)
+			)
+			(justify left bottom)
+		)
+	)
+	(label "FT_PWR_EN"
+		(at 15.9235 9.7157 180)
+		(effects
+			(font
+				(size 1.27 1.27)
+			)
+			(justify right bottom)
+		)
+	)
+	(label "FT_PWR_EN"
+		(at 10.8435 4.6357 180)
+		(effects
+			(font
+				(size 1.27 1.27)
+			)
+			(justify right bottom)
+		)
+	)
+	(label "FT_RESET"
+		(at 56.5635 2.0957 0)
+		(effects
+			(font
+				(size 1.27 1.27)
+			)
+			(justify left bottom)
+		)
+	)
+	(label "FT_PWR_EN"
+		(at 21.0035 14.7957 180)
+		(effects
+			(font
+				(size 1.27 1.27)
+			)
+			(justify right bottom)
+		)
+	)
+	(label "FT_RESET"
+		(at 61.6435 7.1757 0)
+		(effects
+			(font
+				(size 1.27 1.27)
+			)
+			(justify left bottom)
+		)
+	)
+	(label "FT_TXD_EN"
+		(at 10.8435 2.0957 180)
+		(effects
+			(font
+				(size 1.27 1.27)
+			)
+			(justify right bottom)
+		)
+	)
 	(global_label "TXD"
 		(shape input)
@@
 		)
 	)
-	(hierarchical_label "FT_CTS"
-		(shape input)
-		(at 134.62 119.38 0)
-		(effects
-			(font
-				(size 1.27 1.27)
-			)
-			(justify left)
-		)
-	)
 	(hierarchical_label "FT_DRS"
 		(shape input)
@@
 		(effects
 			(font
-				(size 1.27 1.27)
-			)
-			(justify left)
-		)
-	)
-	(hierarchical_label "FT_RST"
-		(shape input)
-		(at 134.62 115.57 0)
-		(effects
-			(font

Commit message: feat: 2-layer stackup, bus net class and schematic cleanup
PCB / project
- Reduce board from 4 layers to 2 (F.Cu / B.Cu) for cheaper fabrication
- Add "bus" net class and reorder net class priorities (bus 0, usb_differential 1, ...)

Schematics
- usb_conector_Ft232: add D+ / D-- labels on the USB mini-B data pair
- ft232: add 10K pull-ups, 100nf decoupling and test points on +3.3VA
- tp_ft232: remove solder jumpers JP1/JP2 (TX_Rpi / RX_Rpi now direct)
- Usb_pic32: add C38 100nf decoupling on +5V
- oled: expand connector J25 from 7 to 8 pins
- mcu / idc / power / zigbee / buttons / cnc_pic32: annotation and net cleanup

docs
- Add USB-Mini-B pinout reference images
Parts:
- removed JP1, JP2: SolderJumper_3_Bridged123, Jumper:SolderJumper-3_P1.3mm_Open_RoundedPad1.0x1.5mm_NumberLabels, symbol Jumper:SolderJumper_3_Bridged123
Changed lines of the file:
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@@
-	(wire
-		(pts
-			(xy 140.97 66.04) (xy 147.32 66.04)
-		)
-		(stroke
-			(width 0)
-			(type default)
-		)
-	)
 	(wire
 		(pts
@@
 	(wire
 		(pts
-			(xy 193.04 66.04) (xy 199.39 66.04)
+			(xy 182.88 69.85) (xy 182.88 66.04)
 		)
 		(stroke
@@
 	(wire
 		(pts
-			(xy 135.89 80.01) (xy 135.89 69.85)
+			(xy 135.89 66.04) (xy 135.89 80.01)
 		)
 		(stroke
@@
 	(wire
 		(pts
-			(xy 124.46 66.04) (xy 130.81 66.04)
+			(xy 124.46 66.04) (xy 135.89 66.04)
 		)
 		(stroke
@@
 		(pts
 			(xy 182.88 77.47) (xy 187.96 77.47)
+		)
+		(stroke
+			(width 0)
+			(type default)
+		)
+	)
+	(wire
+		(pts
+			(xy 187.96 69.85) (xy 182.88 69.85)
 		)
 		(stroke
@@
 				)
 				(justify right)
-			)
-		)
-	)
-	(global_label "TX_Rpi"
-		(shape input)
-		(at 199.39 66.04 0)
-		(fields_autoplaced yes)
-		(effects
-			(font
-				(size 1.27 1.27)
-			)
-			(justify left)
-		)
-		(property "Intersheetrefs" "${INTERSHEET_REFS}"
-			(at 208.5437 66.04 0)
-			(hide yes)
-			(show_name no)
-			(do_not_autoplace no)
-			(effects
-				(font
-					(size 1.27 1.27)
-				)
-				(justify left)
-			)
-		)
-	)
-	(global_label "RX_Rpi"
-		(shape input)
-		(at 147.32 66.04 0)
-		(fields_autoplaced yes)
-		(effects
-			(font
-				(size 1.27 1.27)
-			)
-			(justify left)
-		)
-		(property "Intersheetrefs" "${INTERSHEET_REFS}"
-			(at 156.7761 66.04 0)
-			(hide yes)
-			(show_name no)
-			(do_not_autoplace no)
-			(effects
-				(font
-					(size 1.27 1.27)
-				)
-				(justify left)
 			)
 		)
@@
 	)
 	(symbol
-		(lib_id "Jumper:SolderJumper_3_Bridged123")
-		(at 135.89 66.04 0)
-		(unit 1)
-		(body_style 1)
-		(exclude_from_sim no)
-		(in_bom yes)
-		(on_board yes)
-		(in_pos_files yes)
-		(dnp no)
-		(fields_autoplaced yes)
-		(property "Reference" "JP1"
-			(at 135.89 59.69 0)
-			(show_name no)
-			(do_not_autoplace no)
-			(effects
-				(font
-					(size 1.27 1.27)
-				)
-			)
-		)
-		(property "Value" "SolderJumper_3_Bridged123"
-			(at 135.89 62.23 0)
-			(show_name no)
-			(do_not_autoplace no)
-			(effects
-				(font
-					(size 1.27 1.27)
-				)
-			)
-		)
-		(property "Footprint" "Jumper:SolderJumper-3_P1.3mm_Open_RoundedPad1.0x1.5mm_NumberLabels"
-			(at 135.89 66.04 0)
-			(hide yes)
-			(show_name no)
-			(do_not_autoplace no)
-			(effects
-				(font
-					(size 1.27 1.27)
-				)
-			)
-		)
-		(property "Datasheet" ""
-			(at 135.89 66.04 0)
-			(hide yes)
-			(show_name no)
-			(do_not_autoplace no)
-			(effects
-				(font
-					(size 1.27 1.27)
-				)
-			)
-		)
-		(property "Description" ""
-			(at 135.89 66.04 0)
-			(show_name no)
-			(do_not_autoplace no)
-			(effects
-				(font
-					(size 1.27 1.27)
-				)
-			)
-		)
-		(pin "1"
-		)
-		(pin "2"
-		)
-		(pin "3"
-		)
-		(instances
-			(project "cnc_pic32"
-				(path "/13dbfc1f-be47-44ca-9042-3d6a9a657d7d/22a12b0c-67ed-4f76-a580-7ac736b63dbd/aa6b2b7f-e067-4903-af41-a51929953e3c"
-					(reference "JP1")
-					(unit 1)
-				)
-			)
-		)
-	)
-	(symbol
 		(lib_id "Connector:Conn_01x01_Pin")
 		(at 203.2 115.57 0)
@@
 					(unit 1)
 				)
-			)
-		)
-	)
-	(symbol
-		(lib_id "Jumper:SolderJumper_3_Bridged123")
-		(at 187.96 66.04 0)
-		(unit 1)
-		(body_style 1)
-		(exclude_from_sim no)
-		(in_bom yes)
-		(on_board yes)
-		(in_pos_files yes)
-		(dnp no)
-		(fields_autoplaced yes)
-		(property "Reference" "JP2"
-			(at 187.96 59.69 0)
-			(show_name no)
-			(do_not_autoplace no)
-			(effects
-				(font
-					(size 1.27 1.27)
-				)
-			)
-		)
-		(property "Value" "SolderJumper_3_Bridged123"
-			(at 187.96 62.23 0)
-			(show_name no)
-			(do_not_autoplace no)
-			(effects
-				(font
-					(size 1.27 1.27)
-				)
-			)
-		)
-		(property "Footprint" "Jumper:SolderJumper-3_P1.3mm_Open_RoundedPad1.0x1.5mm_NumberLabels"
-			(at 187.96 66.04 0)
-			(hide yes)
-			(show_name no)
-			(do_not_autoplace no)
-			(effects
-				(font
-					(size 1.27 1.27)
-				)
-			)
-		)
-		(property "Datasheet" ""
-			(at 187.96 66.04 0)
-			(hide yes)
-			(show_name no)
-			(do_not_autoplace no)
-			(effects
-				(font
-					(size 1.27 1.27)
-				)
-			)
-		)
-		(property "Description" ""
-			(at 187.96 66.04 0)
-			(show_name no)
-			(do_not_autoplace no)
-			(effects
-				(font
-					(size 1.27 1.27)
-				)
-			)
-		)
-		(pin "1"
-		)
-		(pin "2"
-		)
-		(pin "3"
-		)
-		(instances
-			(project "cnc_pic32"
-				(path "/13dbfc1f-be47-44ca-9042-3d6a9a657d7d/22a12b0c-67ed-4f76-a580-7ac736b63dbd/aa6b2b7f-e067-4903-af41-a51929953e3c"
-					(reference "JP2")
-					(unit 1)
-				)
