File: tp_ft232.kicad_sch (KiCad schematic)
At the start: 10 parts, among them J10 tp_ft232_, J11 tp_ft232_, J12 tp_ft232_, J16 tp_ft232_, J6 tp_ft232_, J7 tp_ft232_, J8 tp_ft232_, J9 tp_ft232_

Commit message: Clear footprints de KiCad 10 no disponibles en KiCad 7
Parts:
- J10, J11, J12, J6, J7, J8, J9: footprint Connector_Pin:pad_0508 -> (none)
- J16: footprint Connector_Pin:Pin_D1.5mmx1mm -> (none)
Changed lines of the file:
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@@
 			)
 		)
-		(property "Footprint" "Connector_Pin:pad_0508"
+		(property "Footprint" ""
 			(at 123.19 138.43 0)
 			(hide yes)
@@
 			)
 		)
-		(property "Footprint" "Connector_Pin:pad_0508"
+		(property "Footprint" ""
 			(at 118.11 107.95 0)
 			(hide yes)
@@
 			)
 		)
-		(property "Footprint" "Connector_Pin:pad_0508"
+		(property "Footprint" ""
 			(at 118.11 92.71 0)
 			(hide yes)
@@
 			)
 		)
-		(property "Footprint" "Connector_Pin:pad_0508"
+		(property "Footprint" ""
 			(at 118.11 97.79 0)
 			(hide yes)
@@
 			)
 		)
-		(property "Footprint" "Connector_Pin:pad_0508"
+		(property "Footprint" ""
 			(at 124.46 132.08 0)
 			(hide yes)
@@
 			)
 		)
-		(property "Footprint" "Connector_Pin:Pin_D1.5mmx1mm"
+		(property "Footprint" ""
 			(at 203.2 115.57 0)
 			(hide yes)
@@
 			)
 		)
-		(property "Footprint" "Connector_Pin:pad_0508"
+		(property "Footprint" ""
 			(at 118.11 105.41 0)
 			(hide yes)
@@
 			)
 		)
-		(property "Footprint" "Connector_Pin:pad_0508"
+		(property "Footprint" ""
 			(at 118.11 102.87 0)
 			(hide yes)

Commit message: Extraer footprints de example.kicad_pcb y asignarlos a los esquematicos
Parts:
- J10, J11, J12, J6, J7, J8, J9: footprint (none) -> custom:pad_0508
- J16: footprint (none) -> custom:Pin_D1.5mmx1mm
Changed lines of the file:
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@@
 			)
 		)
-		(property "Footprint" ""
+		(property "Footprint" "custom:pad_0508"
 			(at 123.19 138.43 0)
 			(hide yes)
@@
 			)
 		)
-		(property "Footprint" ""
+		(property "Footprint" "custom:pad_0508"
 			(at 118.11 107.95 0)
 			(hide yes)
@@
 			)
 		)
-		(property "Footprint" ""
+		(property "Footprint" "custom:pad_0508"
 			(at 118.11 92.71 0)
 			(hide yes)
@@
 			)
 		)
-		(property "Footprint" ""
+		(property "Footprint" "custom:pad_0508"
 			(at 118.11 97.79 0)
 			(hide yes)
@@
 			)
 		)
-		(property "Footprint" ""
+		(property "Footprint" "custom:pad_0508"
 			(at 124.46 132.08 0)
 			(hide yes)
@@
 			)
 		)
-		(property "Footprint" ""
+		(property "Footprint" "custom:Pin_D1.5mmx1mm"
 			(at 203.2 115.57 0)
 			(hide yes)
@@
 			)
 		)
-		(property "Footprint" ""
+		(property "Footprint" "custom:pad_0508"
 			(at 118.11 105.41 0)
 			(hide yes)
@@
 			)
 		)
-		(property "Footprint" ""
+		(property "Footprint" "custom:pad_0508"
 			(at 118.11 102.87 0)
 			(hide yes)

Commit message: CNC Raspberry update
Parts:
- removed JP1, JP2: SolderJumper_3_Bridged123, Jumper:SolderJumper-3_P1.3mm_Open_RoundedPad1.0x1.5mm_NumberLabels, symbol Jumper:SolderJumper_3_Bridged123
- J10: renamed from J9; footprint custom:pad_0508 -> Library:connector_pin1
- J11: renamed from J10; footprint custom:pad_0508 -> Library:connector_pin1
- J12: renamed from J11; footprint custom:pad_0508 -> Library:connector_pin1
- J13: renamed from J12; footprint custom:pad_0508 -> Library:connector_pin1
- J14: renamed from J16; footprint custom:Pin_D1.5mmx1mm -> Library:connector_pin1
- J7: renamed from J6; footprint custom:pad_0508 -> Library:connector_pin1
- J8: renamed from J7; footprint custom:pad_0508 -> Library:connector_pin1
- J9: renamed from J8; footprint custom:pad_0508 -> Library:connector_pin1
Connections:
- net FT_RTS renamed FT_RST
