File: usb_conector_Ft232.kicad_sch (KiCad schematic)
At the start: 9 parts, among them J15 tp_ft232_, J4 tp_ft232_, J5 USB_B_Mini, U3 LM1117DT-3.3

Commit message: Fix KiCad 10 footprint library: register kiC library, fix schematic references
Parts:
- J15, J4: footprint Connector_Pin:Pin_D1.5mmx1mm -> kiC:Pin_D1.5mmx1mm
Changed lines of the file:
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@@
 			)
 		)
-		(property "Footprint" "Connector_Pin:Pin_D1.5mmx1mm"
+		(property "Footprint" "kiC:Pin_D1.5mmx1mm"
 			(at 156.21 78.74 0)
 			(hide yes)
@@
 			)
 		)
-		(property "Footprint" "Connector_Pin:Pin_D1.5mmx1mm"
+		(property "Footprint" "kiC:Pin_D1.5mmx1mm"
 			(at 114.3 72.39 0)
 			(hide yes)

Commit message: feat: 25 hierarchical labels for 5 Pololus + fix J4/J15/J17/TP17 footprints + USB pin6→SH
- pololu.kicad_sch: 5→25 hierarchical labels (reset_N, sleep_N, enable_N, step_N, dir_N) with wires to each Pololu A4988
- pololu.kicad_sch: J17 footprint kiC:PinHeader → Library:PinHeader_1x06_P2.54mm_Vertical
- cnc_pic32.kicad_sch: expanded Pololu sheet box with 25 named sheet pins
- buttons.kicad_sch: all SW switches → Button_Switch_SMD:SW_SPST_CK_RS282G05A3
- tp_ft232.kicad_sch: kiC:pad_0508 + kiC:Pin_D1.5mmx1mm → Library:connector_pin1
- usb_conector_Ft232.kicad_sch: J4/J15 kiC:Pin_D1.5mmx1mm → Library:connector_pin1, J5 pin 6→SH
- Usb_pic32.kicad_sch: TP17 kiC:Pin_D1.5mmx1mm → Library:connector_pin1, J18 pin 6→SH
Parts:
- J4: footprint kiC:Pin_D1.5mmx1mm -> Library:connector_pin1
- J6: renamed from J15; footprint kiC:Pin_D1.5mmx1mm -> Library:connector_pin1
- renumbered C14 to C19, C15 to C20, L1 to L2, R29 to R28, R30 to R29, U3 to U4
Changed lines of the file:
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@@
 		(dnp no)
 		(fields_autoplaced yes)
-		(property "Reference" "#PWR016"
+		(property "Reference" "#PWR027"
 			(at 123.19 123.19 0)
 			(hide yes)
@@
 			(project "cnc_pic32"
 				(path "/13dbfc1f-be47-44ca-9042-3d6a9a657d7d/22a12b0c-67ed-4f76-a580-7ac736b63dbd/13c6ea59-7a61-4b45-80a4-2330f6dead08"
-					(reference "#PWR016")
+					(reference "#PWR027")
 					(unit 1)
 				)
@@
 		(in_pos_files yes)
 		(dnp no)
-		(property "Reference" "L1"
+		(property "Reference" "L2"
 			(at 144.78 81.28 90)
 			(show_name no)
@@
 			(project "cnc_pic32"
 				(path "/13dbfc1f-be47-44ca-9042-3d6a9a657d7d/22a12b0c-67ed-4f76-a580-7ac736b63dbd/13c6ea59-7a61-4b45-80a4-2330f6dead08"
-					(reference "L1")
+					(reference "L2")
 					(unit 1)
 				)
@@
 		(dnp no)
 		(fields_autoplaced yes)
-		(property "Reference" "#PWR017"
+		(property "Reference" "#PWR028"
 			(at 173.99 106.68 0)
 			(hide yes)
@@
 			(project "cnc_pic32"
 				(path "/13dbfc1f-be47-44ca-9042-3d6a9a657d7d/22a12b0c-67ed-4f76-a580-7ac736b63dbd/13c6ea59-7a61-4b45-80a4-2330f6dead08"
-					(reference "#PWR017")
+					(reference "#PWR028")
 					(unit 1)
 				)
@@
 		(in_pos_files yes)
 		(dnp no)
-		(property "Reference" "R30"
+		(property "Reference" "R29"
 			(at 144.78 93.98 90)
 			(show_name no)
@@
 			(project "cnc_pic32"
 				(path "/13dbfc1f-be47-44ca-9042-3d6a9a657d7d/22a12b0c-67ed-4f76-a580-7ac736b63dbd/13c6ea59-7a61-4b45-80a4-2330f6dead08"
-					(reference "R30")
+					(reference "R29")
 					(unit 1)
 				)
@@
 		(pin "5"
 		)
-		(pin "6"
+		(pin "SH"
 		)
 		(instances
@@
 		(in_pos_files yes)
 		(dnp no)
-		(property "Reference" "J15"
+		(property "Reference" "J6"
 			(at 154.94 77.47 0)
 			(show_name no)
@@
 			)
 		)
-		(property "Footprint" "kiC:Pin_D1.5mmx1mm"
+		(property "Footprint" "Library:connector_pin1"
 			(at 156.21 78.74 0)
 			(hide yes)
@@
 			(project "cnc_pic32"
 				(path "/13dbfc1f-be47-44ca-9042-3d6a9a657d7d/22a12b0c-67ed-4f76-a580-7ac736b63dbd/13c6ea59-7a61-4b45-80a4-2330f6dead08"
-					(reference "J15")
+					(reference "J6")
 					(unit 1)
 				)
@@
 		(in_pos_files yes)
 		(dnp no)
-		(property "Reference" "C15"
+		(property "Reference" "C20"
 			(at 193.802 92.202 0)
 			(show_name no)
@@
 			(project "cnc_pic32"
 				(path "/13dbfc1f-be47-44ca-9042-3d6a9a657d7d/22a12b0c-67ed-4f76-a580-7ac736b63dbd/13c6ea59-7a61-4b45-80a4-2330f6dead08"
-					(reference "C15")
+					(reference "C20")
 					(unit 1)
 				)
@@
 		(dnp no)
 		(fields_autoplaced yes)
-		(property "Reference" "U3"
+		(property "Reference" "U4"
 			(at 173.99 78.74 0)
 			(show_name no)
@@
 			(project "cnc_pic32"
 				(path "/13dbfc1f-be47-44ca-9042-3d6a9a657d7d/22a12b0c-67ed-4f76-a580-7ac736b63dbd/13c6ea59-7a61-4b45-80a4-2330f6dead08"
-					(reference "U3")
+					(reference "U4")
 					(unit 1)
 				)
@@
 		(in_pos_files yes)
 		(dnp no)
-		(property "Reference" "R29"
+		(property "Reference" "R28"
 			(at 144.78 106.68 90)
 			(show_name no)
@@
 			(project "cnc_pic32"
 				(path "/13dbfc1f-be47-44ca-9042-3d6a9a657d7d/22a12b0c-67ed-4f76-a580-7ac736b63dbd/13c6ea59-7a61-4b45-80a4-2330f6dead08"
-					(reference "R29")
+					(reference "R28")
 					(unit 1)
 				)
@@
 		(dnp no)
 		(fields_autoplaced yes)
-		(property "Reference" "#PWR018"
+		(property "Reference" "#PWR029"
 			(at 187.96 81.28 0)
 			(hide yes)
@@
 			(project "cnc_pic32"
 				(path "/13dbfc1f-be47-44ca-9042-3d6a9a657d7d/22a12b0c-67ed-4f76-a580-7ac736b63dbd/13c6ea59-7a61-4b45-80a4-2330f6dead08"
-					(reference "#PWR018")
+					(reference "#PWR029")
 					(unit 1)
 				)
@@
 			)
 		)
-		(property "Footprint" "kiC:Pin_D1.5mmx1mm"
+		(property "Footprint" "Library:connector_pin1"
 			(at 114.3 72.39 0)
 			(hide yes)
@@
 		(in_pos_files yes)
 		(dnp no)
-		(property "Reference" "C14"
+		(property "Reference" "C19"
 			(at 167.132 92.202 0)
 			(show_name no)
@@
 			(project "cnc_pic32"
 				(path "/13dbfc1f-be47-44ca-9042-3d6a9a657d7d/22a12b0c-67ed-4f76-a580-7ac736b63dbd/13c6ea59-7a61-4b45-80a4-2330f6dead08"
-					(reference "C14")
-					(unit 1)
-				)
+					(reference "C19")
+					(unit 1)
+				)

Commit message: fix: pololu.kicad_sch repair - restore A1-A5 symbols, fix dir_5 label, remove orphaned elements
Parts:
- J5: footprint Connector_USB:USB_Mini-B_Wuerth_65100516121_Horizontal -> Library:USB_Mini-B_Wuerth_65100516121_Horizontal
Changed lines of the file:
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@@
 		(dnp no)
 		(fields_autoplaced yes)
-		(property "Reference" "#PWR027"
+		(property "Reference" "#PWR029"
 			(at 123.19 123.19 0)
 			(hide yes)
@@
 			(project "cnc_pic32"
 				(path "/13dbfc1f-be47-44ca-9042-3d6a9a657d7d/22a12b0c-67ed-4f76-a580-7ac736b63dbd/13c6ea59-7a61-4b45-80a4-2330f6dead08"
-					(reference "#PWR027")
+					(reference "#PWR029")
 					(unit 1)
 				)
@@
 		(dnp no)
 		(fields_autoplaced yes)
-		(property "Reference" "#PWR028"
+		(property "Reference" "#PWR030"
 			(at 173.99 106.68 0)
 			(hide yes)
@@
 			(project "cnc_pic32"
 				(path "/13dbfc1f-be47-44ca-9042-3d6a9a657d7d/22a12b0c-67ed-4f76-a580-7ac736b63dbd/13c6ea59-7a61-4b45-80a4-2330f6dead08"
-					(reference "#PWR028")
+					(reference "#PWR030")
 					(unit 1)
 				)
@@
 		(property "Value" "USB_B_Mini"
 			(at 118.11 88.9 0)
-			(show_name no)
-			(do_not_autoplace no)
-			(effects
-				(font
-					(size 1.27 1.27)
-				)
-			)
-		)
-		(property "Footprint" "Connector_USB:USB_Mini-B_Wuerth_65100516121_Horizontal"
+			(hide yes)
+			(show_name no)
+			(do_not_autoplace no)
+			(effects
+				(font
+					(size 1.27 1.27)
+				)
+			)
+		)
+		(property "Footprint" "Library:USB_Mini-B_Wuerth_65100516121_Horizontal"
 			(at 121.92 100.33 0)
 			(hide yes)
@@
 		(pin "5"
 		)
-		(pin "SH"
+		(pin "6"
 		)
 		(instances
@@
 		(dnp no)
 		(fields_autoplaced yes)
-		(property "Reference" "#PWR029"
+		(property "Reference" "#PWR031"
 			(at 187.96 81.28 0)
 			(hide yes)
@@
 			(project "cnc_pic32"
 				(path "/13dbfc1f-be47-44ca-9042-3d6a9a657d7d/22a12b0c-67ed-4f76-a580-7ac736b63dbd/13c6ea59-7a61-4b45-80a4-2330f6dead08"
-					(reference "#PWR029")
-					(unit 1)
-				)
+					(reference "#PWR031")
+					(unit 1)
+				)

Commit message: feat: 2-layer stackup, bus net class and schematic cleanup
PCB / project
- Reduce board from 4 layers to 2 (F.Cu / B.Cu) for cheaper fabrication
- Add "bus" net class and reorder net class priorities (bus 0, usb_differential 1, ...)

Schematics
- usb_conector_Ft232: add D+ / D-- labels on the USB mini-B data pair
- ft232: add 10K pull-ups, 100nf decoupling and test points on +3.3VA
- tp_ft232: remove solder jumpers JP1/JP2 (TX_Rpi / RX_Rpi now direct)
- Usb_pic32: add C38 100nf decoupling on +5V
- oled: expand connector J25 from 7 to 8 pins
- mcu / idc / power / zigbee / buttons / cnc_pic32: annotation and net cleanup

docs
- Add USB-Mini-B pinout reference images
Connections:
- net D--: now reaches J5.2 (D-), R29.2
- net D+: now reaches J5.3 (D+), R28.2
Changed lines of the file:
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@@
+		)
+	)
+	(label "D+"
+		(at 129.54 99.06 0)
+		(effects
+			(font
+				(size 1.27 1.27)
+			)
+			(justify left bottom)
+		)
+	)
+	(label "D--"
+		(at 129.54 101.6 0)
+		(effects
+			(font
+				(size 1.27 1.27)
+			)
+			(justify left bottom)
 		)
 	)
