File: usb_conector_Ft232.kicad_sch (KiCad schematic)
At the start: 9 parts, among them J15 tp_ft232_, J4 tp_ft232_, J5 USB_B_Mini, U3 LM1117DT-3.3

Commit message: Clear footprints de KiCad 10 no disponibles en KiCad 7
Parts:
- J15, J4: footprint Connector_Pin:Pin_D1.5mmx1mm -> (none)
Changed lines of the file:
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@@
 			)
 		)
-		(property "Footprint" "Connector_Pin:Pin_D1.5mmx1mm"
+		(property "Footprint" ""
 			(at 156.21 78.74 0)
 			(hide yes)
@@
 			)
 		)
-		(property "Footprint" "Connector_Pin:Pin_D1.5mmx1mm"
+		(property "Footprint" ""
 			(at 114.3 72.39 0)
 			(hide yes)

Commit message: Extraer footprints de example.kicad_pcb y asignarlos a los esquematicos
Parts:
- J15, J4: footprint (none) -> custom:Pin_D1.5mmx1mm
Changed lines of the file:
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@@
 			)
 		)
-		(property "Footprint" ""
+		(property "Footprint" "custom:Pin_D1.5mmx1mm"
 			(at 156.21 78.74 0)
 			(hide yes)
@@
 			)
 		)
-		(property "Footprint" ""
+		(property "Footprint" "custom:Pin_D1.5mmx1mm"
 			(at 114.3 72.39 0)
 			(hide yes)

Commit message: CNC Raspberry update
Parts:
- J4: footprint custom:Pin_D1.5mmx1mm -> Library:connector_pin1
- J5: footprint Connector_USB:USB_Mini-B_Wuerth_65100516121_Horizontal -> Library:USB_Mini-B_Wuerth_65100516121_Horizontal
- J6: renamed from J15; footprint custom:Pin_D1.5mmx1mm -> Library:connector_pin1
- renumbered C14 to C19, C15 to C20, L1 to L2, R29 to R28, R30 to R29, U3 to U4
Connections:
- net D--: now reaches J5.2 (D-), R29.2
- net D+: now reaches J5.3 (D+), R28.2
