File: Usb_pic32.kicad_sch (KiCad schematic)
At the start: 8 parts, among them J18 USB_B_Mini, U5 LM1117DT-3.3

Commit message: Fix KiCad 10 footprint library: register kiC library, fix schematic references
Parts:
- TP17: footprint Connector_Pin:Pin_D1.5mmx1mm -> kiC:Pin_D1.5mmx1mm
Changed lines of the file:
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@@
 			)
 		)
-		(property "Footprint" "Connector_Pin:Pin_D1.5mmx1mm"
+		(property "Footprint" "kiC:Pin_D1.5mmx1mm"
 			(at 182.88 77.47 0)
 			(hide yes)

Commit message: feat: 25 hierarchical labels for 5 Pololus + fix J4/J15/J17/TP17 footprints + USB pin6→SH
- pololu.kicad_sch: 5→25 hierarchical labels (reset_N, sleep_N, enable_N, step_N, dir_N) with wires to each Pololu A4988
- pololu.kicad_sch: J17 footprint kiC:PinHeader → Library:PinHeader_1x06_P2.54mm_Vertical
- cnc_pic32.kicad_sch: expanded Pololu sheet box with 25 named sheet pins
- buttons.kicad_sch: all SW switches → Button_Switch_SMD:SW_SPST_CK_RS282G05A3
- tp_ft232.kicad_sch: kiC:pad_0508 + kiC:Pin_D1.5mmx1mm → Library:connector_pin1
- usb_conector_Ft232.kicad_sch: J4/J15 kiC:Pin_D1.5mmx1mm → Library:connector_pin1, J5 pin 6→SH
- Usb_pic32.kicad_sch: TP17 kiC:Pin_D1.5mmx1mm → Library:connector_pin1, J18 pin 6→SH
Parts:
- TP1: renamed from TP17; footprint kiC:Pin_D1.5mmx1mm -> Library:connector_pin1
- renumbered C29 to C14, C30 to C15, J18 to J2, L2 to L1, R39 to R8, R40 to R9, U5 to U2
Changed lines of the file:
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@@
 		(dnp no)
 		(fields_autoplaced yes)
-		(property "Reference" "U5"
+		(property "Reference" "U2"
 			(at 200.66 73.66 0)
 			(show_name no)
@@
 			(project "cnc_pic32"
 				(path "/13dbfc1f-be47-44ca-9042-3d6a9a657d7d/71987749-cd9a-4512-bfc9-6de6f65225ef"
-					(reference "U5")
+					(reference "U2")
 					(unit 1)
 				)
@@
 		(in_pos_files yes)
 		(dnp no)
-		(property "Reference" "R40"
+		(property "Reference" "R9"
 			(at 171.45 88.9 90)
 			(show_name no)
@@
 			(project "cnc_pic32"
 				(path "/13dbfc1f-be47-44ca-9042-3d6a9a657d7d/71987749-cd9a-4512-bfc9-6de6f65225ef"
-					(reference "R40")
+					(reference "R9")
 					(unit 1)
 				)
@@
 		(dnp no)
 		(fields_autoplaced yes)
-		(property "Reference" "#PWR043"
+		(property "Reference" "#PWR011"
 			(at 214.63 76.2 0)
 			(hide yes)
@@
 			(project "cnc_pic32"
 				(path "/13dbfc1f-be47-44ca-9042-3d6a9a657d7d/71987749-cd9a-4512-bfc9-6de6f65225ef"
-					(reference "#PWR043")
+					(reference "#PWR011")
 					(unit 1)
 				)
@@
 		(in_pos_files yes)
 		(dnp no)
-		(property "Reference" "L2"
+		(property "Reference" "L1"
 			(at 171.45 76.2 90)
 			(show_name no)
@@
 			(project "cnc_pic32"
 				(path "/13dbfc1f-be47-44ca-9042-3d6a9a657d7d/71987749-cd9a-4512-bfc9-6de6f65225ef"
-					(reference "L2")
+					(reference "L1")
 					(unit 1)
 				)
@@
 		(in_pos_files yes)
 		(dnp no)
-		(property "Reference" "C29"
+		(property "Reference" "C14"
 			(at 193.802 87.122 0)
 			(show_name no)
@@
 			(project "cnc_pic32"
 				(path "/13dbfc1f-be47-44ca-9042-3d6a9a657d7d/71987749-cd9a-4512-bfc9-6de6f65225ef"
-					(reference "C29")
+					(reference "C14")
 					(unit 1)
 				)
@@
 		(dnp no)
 		(fields_autoplaced yes)
-		(property "Reference" "#PWR041"
+		(property "Reference" "#PWR09"
 			(at 149.86 118.11 0)
 			(hide yes)
@@
 			(project "cnc_pic32"
 				(path "/13dbfc1f-be47-44ca-9042-3d6a9a657d7d/71987749-cd9a-4512-bfc9-6de6f65225ef"
-					(reference "#PWR041")
+					(reference "#PWR09")
 					(unit 1)
 				)
@@
 		(in_pos_files yes)
 		(dnp no)
-		(property "Reference" "TP17"
+		(property "Reference" "TP1"
 			(at 181.61 76.2 0)
 			(show_name no)
@@
 			)
 		)
-		(property "Footprint" "kiC:Pin_D1.5mmx1mm"
+		(property "Footprint" "Library:connector_pin1"
 			(at 182.88 77.47 0)
 			(hide yes)
@@
 			(project "cnc_pic32"
 				(path "/13dbfc1f-be47-44ca-9042-3d6a9a657d7d/71987749-cd9a-4512-bfc9-6de6f65225ef"
-					(reference "TP17")
+					(reference "TP1")
 					(unit 1)
 				)
@@
 		(in_pos_files yes)
 		(dnp no)
-		(property "Reference" "R39"
+		(property "Reference" "R8"
 			(at 171.45 101.6 90)
 			(show_name no)
@@
 			(project "cnc_pic32"
 				(path "/13dbfc1f-be47-44ca-9042-3d6a9a657d7d/71987749-cd9a-4512-bfc9-6de6f65225ef"
-					(reference "R39")
+					(reference "R8")
 					(unit 1)
 				)
@@
 		(dnp no)
 		(fields_autoplaced yes)
-		(property "Reference" "J18"
+		(property "Reference" "J2"
 			(at 144.78 81.28 0)
 			(show_name no)
@@
 		(pin "5"
 		)
-		(pin "6"
-		)
-		(instances
-			(project "cnc_pic32"
-				(path "/13dbfc1f-be47-44ca-9042-3d6a9a657d7d/71987749-cd9a-4512-bfc9-6de6f65225ef"
-					(reference "J18")
+		(pin "SH"
+		)
+		(instances
+			(project "cnc_pic32"
+				(path "/13dbfc1f-be47-44ca-9042-3d6a9a657d7d/71987749-cd9a-4512-bfc9-6de6f65225ef"
+					(reference "J2")
 					(unit 1)
 				)
@@
 		(in_pos_files yes)
 		(dnp no)
-		(property "Reference" "C30"
+		(property "Reference" "C15"
 			(at 220.472 87.122 0)
 			(show_name no)
@@
 			(project "cnc_pic32"
 				(path "/13dbfc1f-be47-44ca-9042-3d6a9a657d7d/71987749-cd9a-4512-bfc9-6de6f65225ef"
-					(reference "C30")
+					(reference "C15")
 					(unit 1)
 				)
@@
 		(dnp no)
 		(fields_autoplaced yes)
-		(property "Reference" "#PWR042"
+		(property "Reference" "#PWR010"
 			(at 200.66 101.6 0)
 			(hide yes)
@@
 			(project "cnc_pic32"
 				(path "/13dbfc1f-be47-44ca-9042-3d6a9a657d7d/71987749-cd9a-4512-bfc9-6de6f65225ef"
-					(reference "#PWR042")
-					(unit 1)
-				)
+					(reference "#PWR010")
+					(unit 1)
+				)

Commit message: fix: pololu.kicad_sch repair - restore A1-A5 symbols, fix dir_5 label, remove orphaned elements
Parts:
- J2: footprint Connector_USB:USB_Mini-B_Wuerth_65100516121_Horizontal -> Library:USB_Mini-B_Wuerth_65100516121_Horizontal

Commit message: feat: 2-layer stackup, bus net class and schematic cleanup
PCB / project
- Reduce board from 4 layers to 2 (F.Cu / B.Cu) for cheaper fabrication
- Add "bus" net class and reorder net class priorities (bus 0, usb_differential 1, ...)

Schematics
- usb_conector_Ft232: add D+ / D-- labels on the USB mini-B data pair
- ft232: add 10K pull-ups, 100nf decoupling and test points on +3.3VA
- tp_ft232: remove solder jumpers JP1/JP2 (TX_Rpi / RX_Rpi now direct)
- Usb_pic32: add C38 100nf decoupling on +5V
- oled: expand connector J25 from 7 to 8 pins
- mcu / idc / power / zigbee / buttons / cnc_pic32: annotation and net cleanup

docs
- Add USB-Mini-B pinout reference images
Parts:
- removed TP1: tp_pic+5, Library:connector_pin1, symbol Connector:Conn_01x01_Pin
- added C38: 100nf, Capacitor_SMD:C_1206_3216Metric, symbol Device:C
Connections:
- net GND: now also C38.1
- net +5V: now reaches C14.2, L1.2, U2.3 (VI)
- net +5V: now also C38.2
- net USB_D-: now reaches J2.2 (D-), R9.2
- net USB_D+: now reaches J2.3 (D+), R8.2
Changed lines of the file:
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@@
+	)
+	(junction
+		(at 187.96 90.17)
+		(diameter 0)
+		(color 0 0 0 0)
 	)
 	(junction
@@
 		(color 0 0 0 0)
 	)
+	(junction
+		(at 181.61 80.01)
+		(diameter 0)
+		(color 0 0 0 0)
+	)
 	(wire
 		(pts
@@
 	(wire
 		(pts
+			(xy 181.61 88.9) (xy 181.61 90.17)
+		)
+		(stroke
+			(width 0)
+			(type default)
+		)
+	)
+	(wire
+		(pts
 			(xy 200.66 95.25) (xy 200.66 90.17)
 		)
@@
 	(wire
 		(pts
-			(xy 175.26 80.01) (xy 187.96 80.01)
+			(xy 181.61 90.17) (xy 187.96 90.17)
+		)
+		(stroke
+			(width 0)
+			(type default)
+		)
+	)
+	(wire
+		(pts
+			(xy 175.26 80.01) (xy 181.61 80.01)
 		)
 		(stroke
@@
 	(wire
 		(pts
-			(xy 187.96 77.47) (xy 187.96 80.01)
+			(xy 181.61 81.28) (xy 181.61 80.01)
+		)
+		(stroke
+			(width 0)
+			(type default)
+		)
+	)
+	(wire
+		(pts
+			(xy 181.61 80.01) (xy 187.96 80.01)
 		)
 		(stroke
@@
 			(width 0)
 			(type default)
+		)
+	)
+	(label "D-"
+		(at 173.99 96.52 0)
+		(effects
+			(font
+				(size 1.27 1.27)
+			)
+			(justify left bottom)
+		)
+	)
+	(label "D+"
+		(at 173.99 93.98 0)
+		(effects
+			(font
+				(size 1.27 1.27)
+			)
+			(justify left bottom)
+		)
+	)
+	(label "USB_D+"
+		(at 156.21 93.98 0)
+		(effects
+			(font
+				(size 1.27 1.27)
+			)
+			(justify left bottom)
+		)
+	)
+	(label "USB_D-"
+		(at 156.21 96.52 0)
+		(effects
+			(font
+				(size 1.27 1.27)
+			)
+			(justify left bottom)
 		)
 	)
@@
 	)
 	(symbol
-		(lib_id "Connector:Conn_01x01_Pin")
-		(at 182.88 77.47 0)
-		(mirror x)
+		(lib_id "Device:C")
+		(at 181.61 85.09 180)
 		(unit 1)
 		(body_style 1)
@@
 		(in_pos_files yes)
 		(dnp no)
-		(property "Reference" "TP1"
-			(at 181.61 76.2 0)
-			(show_name no)
-			(do_not_autoplace no)
-			(effects
-				(font
-					(size 1.27 1.27)
-				)
-			)
-		)
-		(property "Value" "tp_pic+5"
-			(at 191.77 76.2 0)
-			(hide yes)
-			(show_name no)
-			(do_not_autoplace no)
-			(effects
-				(font
-					(size 1.27 1.27)
-				)
-			)
-		)
-		(property "Footprint" "Library:connector_pin1"
-			(at 182.88 77.47 0)
+		(property "Reference" "C38"
+			(at 187.452 87.122 0)
+			(show_name no)
+			(do_not_autoplace no)
+			(effects
+				(font
+					(size 1.27 1.27)
+				)
+				(justify left)
+			)
+		)
+		(property "Value" "100nf"
+			(at 188.468 83.058 0)
+			(show_name no)
+			(do_not_autoplace no)
+			(effects
+				(font
+					(size 1.27 1.27)
+				)
+				(justify left)
+			)
+		)
+		(property "Footprint" "Capacitor_SMD:C_1206_3216Metric"
+			(at 180.6448 81.28 0)
 			(hide yes)
 			(show_name no)
@@
 		)
 		(property "Datasheet" ""
-			(at 182.88 77.47 0)
+			(at 181.61 85.09 0)
 			(hide yes)
 			(show_name no)
@@
 		)
 		(property "Description" ""
-			(at 182.88 77.47 0)
+			(at 181.61 85.09 0)
 			(show_name no)
 			(do_not_autoplace no)
@@
 		)
 		(pin "1"
+		)
+		(pin "2"
 		)
 		(instances
 			(project "cnc_pic32"
 				(path "/13dbfc1f-be47-44ca-9042-3d6a9a657d7d/71987749-cd9a-4512-bfc9-6de6f65225ef"
-					(reference "TP1")
+					(reference "C38")
 					(unit 1)
 				)
@@
 					(unit 1)
 				)
+			)
+		)
+	)
+	(symbol
+		(lib_id "power:+5V")
+		(at 181.61 80.01 0)
+		(unit 1)
+		(body_style 1)
+		(exclude_from_sim no)
+		(in_bom yes)
+		(on_board yes)
+		(in_pos_files yes)
+		(dnp no)
+		(fields_autoplaced yes)
+		(property "Reference" "#PWR087"
+			(at 181.61 83.82 0)
+			(hide yes)
+			(show_name no)
+			(do_not_autoplace no)
+			(effects
+				(font
+					(size 1.27 1.27)
+				)
+			)
+		)
+		(property "Value" "+5V"
+			(at 181.61 74.93 0)
+			(show_name no)
+			(do_not_autoplace no)
+			(effects
+				(font
+					(size 1.27 1.27)
+				)
+			)
+		)
+		(property "Footprint" ""
+			(at 181.61 80.01 0)
+			(hide yes)
+			(show_name no)
+			(do_not_autoplace no)
+			(effects
+				(font
+					(size 1.27 1.27)
+				)
+			)
+		)
+		(property "Datasheet" ""
+			(at 181.61 80.01 0)
+			(hide yes)
+			(show_name no)
+			(do_not_autoplace no)
+			(effects
+				(font
+					(size 1.27 1.27)
+				)
+			)
+		)
+		(property "Description" "Power symbol creates a global label with name \"+5V\""
+			(at 181.61 80.01 0)
+			(hide yes)
+			(show_name no)
+			(do_not_autoplace no)
+			(effects
+				(font
+					(size 1.27 1.27)
+				)
+			)
+		)
+		(pin "1"
+		)
+		(instances
+			(project "cnc_pic32"
+				(path "/13dbfc1f-be47-44ca-9042-3d6a9a657d7d/71987749-cd9a-4512-bfc9-6de6f65225ef"
+					(reference "#PWR087")
+					(unit 1)
+				)

Commit message: add files
Parts:
- C14, C15: value 100nf -> 4.7uf
- L1: footprint Inductor_SMD:L_1206_3216Metric -> Inductor_SMD:L_1210_3225Metric
Connections:
- net GND: no longer J2.6 (Shield)
- no-connect marks 0 -> 2
Changed lines of the file:
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@@
-	)
-	(junction
-		(at 144.78 107.95)
-		(diameter 0)
-		(color 0 0 0 0)
 	)
 	(junction
@@
 		(color 0 0 0 0)
 	)
+	(no_connect
+		(at 142.24 107.95)
+	)
+	(no_connect
+		(at 152.4 99.06)
+	)
 	(wire
 		(pts
@@
 		(pts
 			(xy 144.78 107.95) (xy 149.86 107.95)
-		)
-		(stroke
-			(width 0)
-			(type default)
-		)
-	)
-	(wire
-		(pts
-			(xy 142.24 107.95) (xy 144.78 107.95)
 		)
 		(stroke
@@
 			)
 		)
-		(property "Footprint" "Inductor_SMD:L_1206_3216Metric"
+		(property "Footprint" "Inductor_SMD:L_1210_3225Metric"
 			(at 171.45 80.01 0)
 			(hide yes)
@@
 			)
 		)
-		(property "Value" "100nf"
+		(property "Value" "4.7uf"
 			(at 194.818 83.058 0)
 			(show_name no)
@@
 		)
 		(property "Value" "100nf"
-			(at 188.468 83.058 0)
+			(at 180.34 82.804 0)
 			(show_name no)
 			(do_not_autoplace no)
@@
 			)
 		)
-		(property "Value" "100nf"
+		(property "Value" "4.7uf"
 			(at 221.488 83.058 0)
 			(show_name no)

Commit message: updated
Parts:
- J2: now left out of the parts list
Connections:
- net VBUS: now reaches J2.1 (VBUS), L1.1
- net ID: now reaches J2.4 (ID)
- net +5V: no longer names the net of C14.2, C38.2, L1.2, U2.3 (VI)
- no-connect marks 2 -> 1
Changed lines of the file:
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@@
+	)
+	(junction
+		(at 157.48 80.01)
+		(diameter 0)
+		(color 0 0 0 0)
 	)
 	(junction
@@
 		(at 142.24 107.95)
 	)
-	(no_connect
-		(at 152.4 99.06)
-	)
 	(wire
 		(pts
@@
 	(wire
 		(pts
+			(xy 157.48 80.01) (xy 167.64 80.01)
+		)
+		(stroke
+			(width 0)
+			(type default)
+		)
+	)
+	(wire
+		(pts
+			(xy 157.48 73.66) (xy 157.48 80.01)
+		)
+		(stroke
+			(width 0)
+			(type default)
+		)
+	)
+	(wire
+		(pts
 			(xy 177.8 96.52) (xy 172.72 96.52)
 		)
@@
 	(wire
 		(pts
-			(xy 152.4 80.01) (xy 167.64 80.01)
+			(xy 152.4 80.01) (xy 157.48 80.01)
 		)
 		(stroke
@@
 		(pts
 			(xy 181.61 80.01) (xy 187.96 80.01)
+		)
+		(stroke
+			(width 0)
+			(type default)
+		)
+	)
+	(wire
+		(pts
+			(xy 157.48 99.06) (xy 152.4 99.06)
 		)
 		(stroke
@@
 			)
 			(justify left)
+		)
+	)
+	(hierarchical_label "ID"
+		(shape input)
+		(at 157.48 99.06 0)
+		(effects
+			(font
+				(size 1.27 1.27)
+			)
+			(justify left)
+		)
+	)
+	(hierarchical_label "VBUS"
+		(shape input)
+		(at 157.48 73.66 180)
+		(effects
+			(font
+				(size 1.27 1.27)
+			)
+			(justify right)
 		)
 	)
@@
 	)
 	(symbol
+		(lib_id "power:PWR_FLAG")
+		(at 181.61 80.01 0)
+		(unit 1)
+		(body_style 1)
+		(exclude_from_sim no)
+		(in_bom yes)
+		(on_board yes)
+		(in_pos_files yes)
+		(dnp no)
+		(fields_autoplaced yes)
+		(property "Reference" "#FLG04"
+			(at 181.61 78.105 0)
+			(hide yes)
+			(show_name no)
+			(do_not_autoplace no)
+			(effects
+				(font
+					(size 1.27 1.27)
+				)
+			)
+		)
+		(property "Value" "PWR_FLAG"
+			(at 181.61 74.93 0)
+			(show_name no)
+			(do_not_autoplace no)
+			(effects
+				(font
+					(size 1.27 1.27)
+				)
+			)
+		)
+		(property "Footprint" ""
+			(at 181.61 80.01 0)
+			(hide yes)
+			(show_name no)
+			(do_not_autoplace no)
+			(effects
+				(font
+					(size 1.27 1.27)
+				)
+			)
+		)
+		(property "Datasheet" ""
+			(at 181.61 80.01 0)
+			(hide yes)
+			(show_name no)
+			(do_not_autoplace no)
+			(effects
+				(font
+					(size 1.27 1.27)
+				)
+			)
+		)
+		(property "Description" "Special symbol for telling ERC where power comes from"
+			(at 181.61 80.01 0)
+			(hide yes)
+			(show_name no)
+			(do_not_autoplace no)
+			(effects
+				(font
+					(size 1.27 1.27)
+				)
+			)
+		)
+		(pin "1"
+		)
+		(instances
+			(project "cnc_pic32"
+				(path "/13dbfc1f-be47-44ca-9042-3d6a9a657d7d/71987749-cd9a-4512-bfc9-6de6f65225ef"
+					(reference "#FLG04")
+					(unit 1)
+				)
+			)
+		)
+	)
+	(symbol
 		(lib_id "Device:C")
 		(at 181.61 85.09 180)
@@
 		(body_style 1)
 		(exclude_from_sim no)
-		(in_bom yes)
+		(in_bom no)
 		(on_board yes)
 		(in_pos_files yes)
@@
 					(unit 1)
 				)
-			)
-		)
-	)
-	(symbol
-		(lib_id "power:+5V")
-		(at 181.61 80.01 0)
-		(unit 1)
-		(body_style 1)
-		(exclude_from_sim no)
-		(in_bom yes)
-		(on_board yes)
-		(in_pos_files yes)
-		(dnp no)
-		(fields_autoplaced yes)
-		(property "Reference" "#PWR087"
-			(at 181.61 83.82 0)
-			(hide yes)
-			(show_name no)
-			(do_not_autoplace no)
-			(effects
-				(font
-					(size 1.27 1.27)
-				)
-			)
-		)
-		(property "Value" "+5V"
-			(at 181.61 74.93 0)
-			(show_name no)
-			(do_not_autoplace no)
-			(effects
-				(font
-					(size 1.27 1.27)
-				)
-			)
-		)
-		(property "Footprint" ""
-			(at 181.61 80.01 0)
-			(hide yes)
-			(show_name no)
-			(do_not_autoplace no)
-			(effects
-				(font
-					(size 1.27 1.27)
-				)
-			)
-		)
-		(property "Datasheet" ""
-			(at 181.61 80.01 0)
-			(hide yes)
-			(show_name no)
-			(do_not_autoplace no)
-			(effects
-				(font
-					(size 1.27 1.27)
-				)
-			)
-		)
-		(property "Description" "Power symbol creates a global label with name \"+5V\""
-			(at 181.61 80.01 0)
-			(hide yes)
-			(show_name no)
-			(do_not_autoplace no)
-			(effects
-				(font
-					(size 1.27 1.27)
-				)
-			)
-		)
-		(pin "1"
-		)
-		(instances
-			(project "cnc_pic32"
-				(path "/13dbfc1f-be47-44ca-9042-3d6a9a657d7d/71987749-cd9a-4512-bfc9-6de6f65225ef"
-					(reference "#PWR087")
-					(unit 1)
-				)
