File: Usb_pic32.kicad_sch (KiCad schematic)
At the start: 8 parts, among them J18 USB_B_Mini, U5 LM1117DT-3.3

Commit message: Clear footprints de KiCad 10 no disponibles en KiCad 7
Parts:
- TP17: footprint Connector_Pin:Pin_D1.5mmx1mm -> (none)
Changed lines of the file:
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@@
 			)
 		)
-		(property "Footprint" "Connector_Pin:Pin_D1.5mmx1mm"
+		(property "Footprint" ""
 			(at 182.88 77.47 0)
 			(hide yes)

Commit message: Extraer footprints de example.kicad_pcb y asignarlos a los esquematicos
Parts:
- TP17: footprint (none) -> custom:Pin_D1.5mmx1mm
Changed lines of the file:
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@@
 			)
 		)
-		(property "Footprint" ""
+		(property "Footprint" "custom:Pin_D1.5mmx1mm"
 			(at 182.88 77.47 0)
 			(hide yes)

Commit message: CNC Raspberry update
Parts:
- removed TP17: tp_pic+5, custom:Pin_D1.5mmx1mm, symbol Connector:Conn_01x01_Pin
- added C38: 100nf, Capacitor_SMD:C_1206_3216Metric, symbol Device:C
- C14: renamed from C29; value 100nf -> 4.7uf
- C15: renamed from C30; value 100nf -> 4.7uf
- J2: renamed from J18; footprint Connector_USB:USB_Mini-B_Wuerth_65100516121_Horizontal -> Library:USB_Mini-B_Wuerth_65100516121_Horizontal; now left out of the parts list
- L1: renamed from L2; footprint Inductor_SMD:L_1206_3216Metric -> Inductor_SMD:L_1210_3225Metric
- renumbered R39 to R8, R40 to R9, U5 to U2
Connections:
- net GND: now also C38.1; no longer J2.6 (Shield)
- net at C14.2, L1.2, U2.3 (VI): now also C38.2
- net USB_D-: now reaches J2.2 (D-), R9.2
- net VBUS: now reaches J2.1 (VBUS), L1.1
- net USB_D+: now reaches J2.3 (D+), R8.2
- net ID: now reaches J2.4 (ID)
- no-connect marks 0 -> 1
