File: ft232.kicad_sch (KiCad schematic)
At the start: 59 parts, among them J10 tp, J11 tp, J12 tp, J13 FT232RL, J14 tp_ft232_, J22 USB_B_Mini, J26 tp_ft232_, J3 tp, J4 tp, J5 tp, J6 tp, J7 tp, J8 tp, J9 tp, Q1 FDN306P, Q2 2N7002, Q3 2N7002, U3 FT232BM, U4 93CxxA, U6 LM1117DT-3.3, Y2 Crystal

Commit message: updated
Parts:
- removed J9: tp, TestPoint:TestPoint_Pad_D1.5mm, symbol Connector:Conn_01x01_Pin
- removed Q2, Q3: 2N7002, Package_TO_SOT_SMD:SOT-23, symbol Transistor_FET:2N7002
- removed R2, R3, R4, R5: 2k2, Resistor_SMD:R_0805_2012Metric, symbol Device:R
- added X2: TAXM8M4RDBCCT2T, Crystal:Crystal_SMD_3225-4Pin_3.2x2.5mm, symbol JLCImport:TAXM8M4RDBCCT2T
- C18, C21: footprint Capacitor_SMD:C_0805_2012Metric -> Capacitor_SMD:C_0603_1608Metric
- C30, C37: value 100nf -> 4.7uf
- D1, D2, J10, J11, J13, J14, J26, J3, J4, J5, J6, J7, J8, JP1, JP2, U3, U4: now left out of the parts list
- J12: footprint TestPoint:TestPoint_THTPad_1.5x1.5mm_Drill0.7mm -> TestPoint:TestPoint_Pad_D1.5mm; now left out of the parts list
- J22: value USB_B_Mini -> Mini-B Surface Mount, Right Angle USB 2.0 SMD USB Connectors ROHS; LCSC (none) -> C91144
- JP24: footprint (none) -> Jumper:SolderJumper-2_P1.3mm_Bridged2Bar_RoundedPad1.0x1.5mm; now left out of the parts list
- R29, R30: value 27 -> 22
- Y2: value Crystal -> Crystal 6MHZ
Connections:
- net FT_XTIN: now also X2.1
- net FT_XTOUT: now also X2.3
- net GND: now also X2.2, X2.4
- net FT_DRS renamed FT_DSR
