File: ft232.kicad_sch (KiCad schematic)
At the start: 20 parts, among them J3 tp_ft232_, Q1 2N7002, U2 FT232BM

Commit message: Clear footprints de KiCad 10 no disponibles en KiCad 7
Parts:
- J3: footprint Connector_Pin:pad_0508 -> (none)
Changed lines of the file:
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@@
 			)
 		)
-		(property "Footprint" "Connector_Pin:pad_0508"
+		(property "Footprint" ""
 			(at 172.72 66.04 0)
 			(hide yes)

Commit message: Extraer footprints de example.kicad_pcb y asignarlos a los esquematicos
Parts:
- J3: footprint (none) -> custom:pad_0508
Changed lines of the file:
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@@
 			)
 		)
-		(property "Footprint" ""
+		(property "Footprint" "custom:pad_0508"
 			(at 172.72 66.04 0)
 			(hide yes)

Commit message: CNC Raspberry update
Parts:
- removed C11: 100nf, Capacitor_SMD:C_0805_2012Metric, symbol Device:C
- removed C12, C13: 33nf, Capacitor_SMD:C_0805_2012Metric, symbol Device:C
- removed Q1: 2N7002, Package_TO_SOT_SMD:SOT-23, symbol Transistor_FET:2N7002
- removed U2: FT232BM, Package_QFP:LQFP-32_7x7mm_P0.8mm, symbol Interface_USB:FT232BM
- added C16, C17, C19, C20, C22: 100nf, Capacitor_SMD:C_0805_2012Metric, symbol Device:C
- added C18, C21: 100nf, Capacitor_SMD:C_0603_1608Metric, symbol Device:C
- added C23, C25: 15p, Capacitor_SMD:C_0805_2012Metric, symbol Device:C
- added C24, C26: 33nf, Capacitor_SMD:C_0805_2012Metric, symbol Device:C
- added C30, C37: 4.7uf, Capacitor_SMD:C_0805_2012Metric, symbol Device:C
- added J10, J11, J12, J4, J5, J6, J7, J8: tp, TestPoint:TestPoint_Pad_D1.5mm, symbol Connector:Conn_01x01_Pin
- added J13: FT232RL, Connector_PinHeader_2.54mm:PinHeader_1x06_P2.54mm_Vertical, symbol Connector:Conn_01x06_Pin
- added J14, J26: tp_ft232_, Library:connector_pin1, symbol Connector:Conn_01x01_Pin
- added J22: Mini-B Surface Mount, Right Angle USB 2.0 SMD USB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, kiC:USB_Mini-B_Lumberg_2486_01_Horizontal, symbol Connector:USB_B_Mini
- added JP1, JP2: Jumper_Open, Jumper:SolderJumper-2_P1.3mm_Open_RoundedPad1.0x1.5mm, symbol Jumper:Jumper_2_Open
- added JP24: Jumper_2_Bridged, Jumper:SolderJumper-2_P1.3mm_Bridged2Bar_RoundedPad1.0x1.5mm, symbol Jumper:Jumper_2_Bridged
- added L2: 100mh, Inductor_SMD:L_1206_3216Metric, symbol Device:L
- added Q1: FDN306P, Package_TO_SOT_SMD:SOT-23W, symbol FDN306P:FDN306P
- added R16: 10K, Resistor_SMD:R_0805_2012Metric, symbol Device:R
- added R29, R30: 22, Resistor_SMD:R_0805_2012Metric, symbol Device:R
- added U3: FT232BM, Package_QFP:LQFP-32_7x7mm_P0.8mm, symbol Interface_USB:FT232BM
- added U4: 93CxxA, Package_SO:SOIC-8_5.3x5.3mm_P1.27mm, symbol Memory_EEPROM:93CxxA
- added U6: LM1117DT-3.3, kiC:SOT-223-3_TabPin2, symbol Regulator_Linear:LM1117DT-3.3
- added X2: TAXM8M4RDBCCT2T, Crystal:Crystal_SMD_3225-4Pin_3.2x2.5mm, symbol JLCImport:TAXM8M4RDBCCT2T
- added Y2: Crystal 6MHZ, Crystal:Resonator-2Pin_W10.0mm_H5.0mm, symbol Device:Crystal
- D1, D2: now left out of the parts list
- J3: value tp_ft232_ -> tp; footprint custom:pad_0508 -> TestPoint:TestPoint_Pad_D1.5mm; now left out of the parts list
- R17: footprint Resistor_SMD:R_0805_2012Metric -> Resistor_SMD:R_0603_1608Metric
- R19, R20: value 10K -> 100
- R21, R22: value 100 -> 10K
- R23, R24: value 10K -> 1K5
- R25: value 1K5 -> 10K
- R27: value 1K5 -> 4K7
- R28: value 4K7 -> 2k2
Connections:
- net FT is gone; now on an unnamed net: R18.2
- net RX_MCU is gone; now on an unnamed net: R21.2
- net FT_CTS: now also C22.2, J13.5 (Pin_5), J4.1 (Pin_1), U3.22 (D3/~{CTS})
- net FT_DCD: now also J7.1 (Pin_1), U3.19 (D6/~{DCD})
- net FT_DTR: now also J13.1 (Pin_1), J5.1 (Pin_1), U3.21 (D4/~{DTR})
- net FT_EECS: now also U3.32 (EECS), U4.1 (CS)
- net FT_EEDATA: now also R28.1, U3.2 (EEDATA), U4.3 (DI)
- net FT_EESK: now also U3.1 (EESK), U4.2 (SCLK)
- net FT_PWR_EN: now also R17.2, J11.1 (Pin_1), U3.15 (~{PWREN}); no longer R19.1
- net FT_RESET: now also R25.2, R27.2, U3.4 (~{RESET}); no longer R28.2
- net FT_RI: now also J8.1 (Pin_1), U3.18 (D7/~{RI})
- net FT_RST: now also J3.1 (Pin_1), U3.23 (D2/~{RST})
- net FT_RST_OUT: now also R24.1, U3.5 (~{RSTOUT}); no longer R27.1
- net FT_TXD_EN: now also J10.1 (Pin_1), U3.16 (TXDEN)
- net FT_USB_DP: now also R24.2, R29.1, U3.7 (USBDP); no longer R27.2
- net FT_XTIN: now also C23.1, U3.27 (XTIN), X2.1, Y2.1
- net FT_XTOUT: now also C25.1, U3.28 (XTOUT), X2.3, Y2.2
- net GND: now also C16.2, C17.2, C19.1, C20.1, C21.1, C23.2, C24.2, C25.2, C26.2, C30.1, C37.1, J13.6 (Pin_6), J22.6 (Shield), JP24.2 (B), R16.1, U3.17 (GND1), U3.29 (AGND1), U3.31 (TEST), U3.9 (GND1), U4.5 (GND1), U6.1 (GND1), X2.2, X2.4; no longer R18.1
- net at D2.1 (K): now also U3.11 (~{RXLED})
- net at D1.1 (K): now also U3.12 (~{TXLED})
- net +3.3VA: now reaches R22.1
- net +3.3VA: now also R18.1, R21.1, R25.1, C16.1, C17.1, C19.2, C20.2, C37.2, U3.13 (VCCIO), U4.8 (VCC), U6.2 (VO)
- net _TX: now reaches R19.2
- net _TX: now also JP1.2 (B)
- net at R17.1: now also C18.1, Q1.1
- net at D2.2 (A): no longer R23.2
- net at D1.2 (A): no longer R20.2
- removed net +3V3: R20.1, R23.1, R24.1
- net TX_MCU: no longer names the net of R22.2
- net TX_MCU: now also U3.10 (~{SLEEP})
- removed net V+_USB: R17.2, R25.2, R28.1
- new net: J22.1 (VBUS), L2.1
- new net: R20.1, U3.24 (D1/RXD)
- new net: R19.1, U3.25 (D0/TXD)
- new net: C24.1, R23.1, U3.30 (AVCC)
- new net: C26.1, J14.1 (Pin_1), U3.6 (3V3OUT)
- new net: J22.3 (D+), R29.2
- new net: J22.2 (D-), R30.2
- new net: R28.2, U4.4 (DO)
- new net: J22.5 (GND1), JP24.1 (A)
- new net +5VA: C18.2, C21.2, C30.2, J13.4 (Pin_4), J26.1 (Pin_1), L2.2, Q1.2, R23.2, R27.1, U3.26 (VCC), U3.3 (VCC), U6.3 (VI)
- new net FT_CTL: R16.2, U3.14 (PWRCTL)
- new net FT_DSR: J6.1 (Pin_1), U3.20 (D5/~{DSR})
- new net FT_RX: J13.3 (Pin_3), JP2.1 (A)
- new net FT_TX: J13.2 (Pin_2), JP1.1 (A)
- new net FT_USB_DM: R30.1, U3.8 (USBDM)
- new net ID: J22.4 (ID)
- new net MCLR: C22.1
- new net PWR: J12.1 (Pin_1), Q1.3
- new net _RX: JP2.2 (B), R20.2
Other:
- removed sheet osc_ft232
- removed sheet power_ft232
- removed sheet tp_ft232
- removed sheet usb_conector_Ft232
- note added: "DTR RTS -> EN IO9 1 1 1 1 0 0 1 1 1 0 0 1 0 1 1 0"
