File: MA240011.kicad_sch (KiCad schematic)
At the start: 14 parts, among them J1 icd, U7 PIC32MX795F512L-80x-PF, Y1 8MHZ

Commit message: add files
Parts:
- removed JP5: pgc1, Jumper:SolderJumper-2_P1.3mm_Open_RoundedPad1.0x1.5mm, symbol Jumper:Jumper_2_Bridged
- removed JP6: pgd1, Jumper:SolderJumper-2_P1.3mm_Open_RoundedPad1.0x1.5mm, symbol Jumper:Jumper_2_Bridged
- removed JP7: pgc2, Jumper:SolderJumper-2_P1.3mm_Bridged_RoundedPad1.0x1.5mm, symbol Jumper:Jumper_2_Bridged
- removed JP8: pgd2, Jumper:SolderJumper-2_P1.3mm_Bridged_RoundedPad1.0x1.5mm, symbol Jumper:Jumper_2_Bridged
- added R42: 0, Resistor_SMD:R_0805_2012Metric, symbol Device:R
- JP3, JP4: footprint (none) -> Jumper:SolderJumper-2_P1.3mm_Open_RoundedPad1.0x1.5mm
Connections:
- net VBUS: now also R42.2; no longer U7.54 (VBUS)
- new net: R42.1, U7.54 (VBUS)

Commit message: updated
Parts:
- removed JP3: sda_jp, Jumper:SolderJumper-2_P1.3mm_Open_RoundedPad1.0x1.5mm, symbol Jumper:Jumper_2_Bridged
- removed JP4: scl_jp, Jumper:SolderJumper-2_P1.3mm_Open_RoundedPad1.0x1.5mm, symbol Jumper:Jumper_2_Bridged
- J1: footprint Connector_PinHeader_2.54mm:PinHeader_1x06_P2.54mm_Horizontal -> Connector_PinHeader_2.54mm:PinHeader_1x06_P2.54mm_Vertical; now left out of the parts list
- R42: footprint Resistor_SMD:R_0805_2012Metric -> Resistor_SMD:R_0603_1608Metric
- U7: now left out of the parts list
- Y1: value 8MHZ -> 8MHz SMD crystal oscillator ±10ppm ±30ppm SMD3225-4P Crystals; footprint Crystal:Crystal_SMD_0603-4Pin_6.0x3.5mm -> Crystal:Crystal_SMD_3225-4Pin_3.2x2.5mm; LCSC (none) -> C20617233
Connections:
- net RD14 renamed RD14_SS3_U4RX
- net RF12 renamed RF12_SS4
- net RF13 renamed RF13_SCK4
- net RF4 renamed RF4_SDO4
- net RF5 renamed RF5_SDI4

Commit message: LPCXpresso
Parts:
- removed C11: 100nf, Capacitor_SMD:C_0805_2012Metric, symbol Device:C
- removed C12, C13: 15p, Capacitor_SMD:C_0805_2012Metric, symbol Device:C
- removed J1: icd, Connector_PinHeader_2.54mm:PinHeader_1x06_P2.54mm_Vertical, symbol Connector:Conn_01x06_Pin
- removed R6: 1K, Resistor_SMD:R_0805_2012Metric, symbol Device:R
- removed R7: 1M, Resistor_SMD:R_0805_2012Metric, symbol Device:R
- removed Y1: 8MHz SMD crystal oscillator ±10ppm ±30ppm SMD3225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, Crystal:Crystal_SMD_3225-4Pin_3.2x2.5mm, symbol Device:Crystal_GND24
- U7: now not fitted
