File: cnc_pic32.kicad_pcb (KiCad board)
At the start: 2 copper layers, 96 x 96 mm, 164 parts, among them J1 icd, J10 tp, J11 tp, J12 tp, J13 FT232RL, J15 pololu, J16 pololu, J17 pololu, J18 pololu, J19 pololu, J2 USB_B_Mini, J20 pololu, J21 conector oled ST1306 128x32, J22 USB_B_Mini, J23 Conn_01x04_Pin, J25 Conn_01x08_Pin, J3 tp, J4 tp, J5 tp, J6 tp, J7 tp, J8 tp, J9 tp, Q1 FDN306P, Q2 2N7002, Q3 2N7002, SW1 power, SW2 up, SW3 down, SW4 left, SW5 rigth, U1 PIC32MX795F512L-80x-PF, U2 LM1117DT-3.3, U3 FT232BM, U4 93CxxA, U6 LM1117DT-3.3, U7 PIC32MX795F512L-80x-PF, U8 ESP8266-12E_ESP-12E, Y1 8MHZ, Y2 Crystal

Commit message: updated
Parts:
- removed C46: 10uf, Capacitor_SMD:C_Elec_6.3x5.4
- removed J16: pololu, Library:PinHeader_1x06_P2.54mm_Vertical
- removed J9: tp, TestPoint:TestPoint_Pad_D1.5mm
- removed JP3: sda_jp, Jumper:SolderJumper-2_P1.3mm_Open_RoundedPad1.0x1.5mm
- removed JP4: scl_jp, Jumper:SolderJumper-2_P1.3mm_Open_RoundedPad1.0x1.5mm
- removed Q2, Q3: 2N7002, Package_TO_SOT_SMD:SOT-23
- removed R2, R4, R5: 2k2, Resistor_SMD:R_0805_2012Metric
- added A10: Pololu_Breakout_DRV8825, kiC:HTSSOP-28-EP_IC_TPS61196PWPRQ1, F.Cu at (132.7, 93.7)
- added A6: Pololu_Breakout_DRV8825, kiC:HTSSOP-28-EP_IC_TPS61196PWPRQ1, F.Cu at (132.4, 56.3)
- added A7: Pololu_Breakout_DRV8825, kiC:HTSSOP-28-EP_IC_TPS61196PWPRQ1, F.Cu at (132.3, 38.7)
- added A8: Pololu_Breakout_DRV8825, kiC:HTSSOP-28-EP_IC_TPS61196PWPRQ1, F.Cu at (132.7, 73.9)
- added A9: Pololu_Breakout_DRV8825, kiC:HTSSOP-28-EP_IC_TPS61196PWPRQ1, F.Cu at (133.1, 112.3)
- added C51: EFVH035ADA100M0454, Capacitor_SMD:C_Elec_5x5.4, F.Cu at (118.1, 47.5)
- added C52: EFVH035ADA100M0454, Capacitor_SMD:C_Elec_5x5.4, F.Cu at (117.4, 64.9)
- added C53: 100nf, Capacitor_SMD:C_0805_2012Metric, F.Cu at (140.0, 52.5)
- added C54: 100nf, Capacitor_SMD:C_0805_2012Metric, F.Cu at (140.5, 70.3)
- added C55: 100nf, Capacitor_SMD:C_0805_2012Metric, F.Cu at (140.2, 89.9)
- added C56: 100nf, Capacitor_SMD:C_0805_2012Metric, F.Cu at (140.3, 108.4)
- added C57: 100nf, Capacitor_SMD:C_0805_2012Metric, F.Cu at (124.8, 52.6)
- added C58: 100nf, Capacitor_SMD:C_0805_2012Metric, F.Cu at (124.9, 70.5)
- added C59: 100nf, Capacitor_SMD:C_0805_2012Metric, F.Cu at (125.0, 90.0)
- added C60: 100nf, Capacitor_SMD:C_0805_2012Metric, F.Cu at (125.2, 108.6)
- added D6: LED, Diode_SMD:D_0805_2012Metric, F.Cu at (89.9, 51.7)
- added D7: LED, Diode_SMD:D_0805_2012Metric, F.Cu at (87.5, 51.7)
- added D8: LED, Diode_SMD:D_0805_2012Metric, F.Cu at (85.2, 51.7)
- added J24: Micro_SD_Card, JLCImport:TF-001B, F.Cu at (102.6, 113.6)
- added JP24: Jumper_2_Bridged, Jumper:SolderJumper-2_P1.3mm_Bridged2Bar_RoundedPad1.0x1.5mm, B.Cu at (59.5, 115.8)
- added JP25: MS3, Jumper:SolderJumper-2_P1.3mm_Open_RoundedPad1.0x1.5mm, B.Cu at (140.4, 34.8)
- added JP26: MS3, Jumper:SolderJumper-2_P1.3mm_Open_RoundedPad1.0x1.5mm, B.Cu at (140.4, 37.4)
- added JP27: MS3, Jumper:SolderJumper-2_P1.3mm_Open_RoundedPad1.0x1.5mm, B.Cu at (140.4, 40.0)
- added JP28: MS3, Jumper:SolderJumper-2_P1.3mm_Open_RoundedPad1.0x1.5mm, B.Cu at (140.4, 42.6)
- added JP29: MS3, Jumper:SolderJumper-2_P1.3mm_Open_RoundedPad1.0x1.5mm, B.Cu at (139.5, 52.4)
- added JP30: MS3, Jumper:SolderJumper-2_P1.3mm_Open_RoundedPad1.0x1.5mm, B.Cu at (139.5, 55.3)
- added JP31: MS3, Jumper:SolderJumper-2_P1.3mm_Open_RoundedPad1.0x1.5mm, B.Cu at (139.5, 57.9)
- added JP32: MS3, Jumper:SolderJumper-2_P1.3mm_Open_RoundedPad1.0x1.5mm, B.Cu at (139.5, 60.7)
- added JP33: MS3, Jumper:SolderJumper-2_P1.3mm_Open_RoundedPad1.0x1.5mm, B.Cu at (141.4, 89.7)
- added JP34: MS3, Jumper:SolderJumper-2_P1.3mm_Open_RoundedPad1.0x1.5mm, B.Cu at (141.4, 92.3)
- added JP35: MS3, Jumper:SolderJumper-2_P1.3mm_Open_RoundedPad1.0x1.5mm, B.Cu at (141.4, 95.3)
- added JP36: MS3, Jumper:SolderJumper-2_P1.3mm_Open_RoundedPad1.0x1.5mm, B.Cu at (141.4, 97.6)
- added JP37: MS3, Jumper:SolderJumper-2_P1.3mm_Open_RoundedPad1.0x1.5mm, B.Cu at (140.9, 108.2)
- added JP38: MS3, Jumper:SolderJumper-2_P1.3mm_Open_RoundedPad1.0x1.5mm, B.Cu at (140.9, 110.7)
- added JP39: MS3, Jumper:SolderJumper-2_P1.3mm_Open_RoundedPad1.0x1.5mm, B.Cu at (140.9, 113.4)
- added JP40: MS3, Jumper:SolderJumper-2_P1.3mm_Open_RoundedPad1.0x1.5mm, B.Cu at (140.9, 116.1)
- added JP41: MS3, Jumper:SolderJumper-2_P1.3mm_Open_RoundedPad1.0x1.5mm, B.Cu at (140.6, 70.3)
- added JP42: MS3, Jumper:SolderJumper-2_P1.3mm_Open_RoundedPad1.0x1.5mm, B.Cu at (140.6, 73.0)
- added JP43: MS3, Jumper:SolderJumper-2_P1.3mm_Open_RoundedPad1.0x1.5mm, B.Cu at (140.6, 75.4)
- added JP44: MS3, Jumper:SolderJumper-2_P1.3mm_Open_RoundedPad1.0x1.5mm, B.Cu at (140.5, 77.8)
- added R44: 2k2, Resistor_SMD:R_0805_2012Metric, F.Cu at (96.8, 103.1)
- added R45: 2k2, Resistor_SMD:R_0805_2012Metric, F.Cu at (99.8, 102.7)
- added R46: 2k2, Resistor_SMD:R_0805_2012Metric, F.Cu at (102.3, 102.6)
- added R47: 2k2, Resistor_SMD:R_0805_2012Metric, F.Cu at (105.0, 102.7)
- added R48: 2k2, Resistor_SMD:R_0805_2012Metric, F.Cu at (107.8, 102.7)
- added R49: 2k2, Resistor_SMD:R_0805_2012Metric, F.Cu at (94.6, 103.0)
- added R50: 1k, Resistor_SMD:R_0805_2012Metric, F.Cu at (87.6, 56.1)
- added R51: 1k, Resistor_SMD:R_0805_2012Metric, F.Cu at (85.4, 56.1)
- added X2: TAXM8M4RDBCCT2T, Crystal:Crystal_SMD_3225-4Pin_3.2x2.5mm, F.Cu at (72.6, 104.9)
- C10, C27, C28, C3, C4, C9: footprint Capacitor_SMD:C_0805_2012Metric -> Resistor_SMD:R_0603_1608Metric
- C16, C17, C19, C20, C22, C23, C25, J13, Q1, R16, R17, R22, R25, R26, R27, R28: moved to B.Cu
- C18, C21: footprint Capacitor_SMD:C_0805_2012Metric -> Capacitor_SMD:C_0603_1608Metric; moved to B.Cu
- C30, C37: value 100nf -> 4.7uf; moved to B.Cu
- C36: value 100nf -> 4.7uf
- C39, C40, C41, C48, C49, C50: value 10uf -> RVT100UF35V67RV0034
- C42, C43, C45, C47: value 10uf -> EFVH035ADA100M0454; footprint Capacitor_SMD:C_Elec_6.3x5.4 -> Capacitor_SMD:C_Elec_5x5.4
- C44: value 10uf -> 100nf; footprint Capacitor_SMD:C_Elec_6.3x5.4 -> Capacitor_SMD:C_0805_2012Metric
- J1: footprint Connector_PinHeader_2.54mm:PinHeader_1x06_P2.54mm_Horizontal -> Connector_PinHeader_2.54mm:PinHeader_1x06_P2.54mm_Vertical
- J12: footprint TestPoint:TestPoint_THTPad_1.5x1.5mm_Drill0.7mm -> TestPoint:TestPoint_Pad_D1.5mm; moved to B.Cu
- J22: value USB_B_Mini -> Mini-B Surface Mount, Right Angle USB 2.0 SMD USB Connectors ROHS
- J23: value Conn_01x04_Pin -> OLED SSD1306
- J25: footprint Library:Adafruit_SSD1306_No_Mounting_Holes_pads -> Connector_PinHeader_2.54mm:PinHeader_1x08_P2.54mm_Vertical
- R29, R30: value 27 -> 22
- R3: value 2k2 -> 1k
- R42, R43: footprint Resistor_SMD:R_0805_2012Metric -> Resistor_SMD:R_0603_1608Metric
- SW1: value power -> K2-1107ST-A4SW-06; footprint Button_Switch_SMD:SW_SPST_CK_RS282G05A3 -> Button_Switch_SMD:SW_Tactile_SPST_NO_Straight_CK_PTS636Sx25SMTRLFS
- SW2: value up -> K2-1107ST-A4SW-06; footprint Button_Switch_SMD:SW_SPST_CK_RS282G05A3 -> Button_Switch_SMD:SW_Tactile_SPST_NO_Straight_CK_PTS636Sx25SMTRLFS
- SW3: value down -> K2-1107ST-A4SW-06; footprint Button_Switch_SMD:SW_SPST_CK_RS282G05A3 -> Button_Switch_SMD:SW_Tactile_SPST_NO_Straight_CK_PTS636Sx25SMTRLFS
- SW4: value left -> K2-1107ST-A4SW-06; footprint Button_Switch_SMD:SW_SPST_CK_RS282G05A3 -> Button_Switch_SMD:SW_Tactile_SPST_NO_Straight_CK_PTS636Sx25SMTRLFS
- SW5: value rigth -> K2-1107ST-A4SW-06; footprint Button_Switch_SMD:SW_SPST_CK_RS282G05A3 -> Button_Switch_SMD:SW_Tactile_SPST_NO_Straight_CK_PTS636Sx25SMTRLFS
- Y1: value 8MHZ -> 8MHz SMD crystal oscillator ±10ppm ±30ppm SMD3225-4P Crystals; footprint Crystal:Crystal_SMD_0603-4Pin_6.0x3.5mm -> Crystal:Crystal_SMD_3225-4Pin_3.2x2.5mm
- Y2: value Crystal -> Crystal 6MHZ; moved to B.Cu
- moved C47 104.4 mm to (70.4, 49.9), turned to -90 degrees
- moved C45 84.2 mm to (117.4, 103.3), turned to -90 degrees
- moved C29 78.1 mm to (139.4, 38.9), turned to -90 degrees
- moved C36 62.6 mm to (83.3, 41.6)
- moved R14 62.4 mm to (56.1, 93.0), turned to -90 degrees
- moved R15 59.1 mm to (56.6, 87.9), turned to -90 degrees
- moved C31 58.0 mm to (124.9, 34.9), turned to 0 degrees
- moved C11 57.8 mm to (54.4, 79.5), turned to -90 degrees
- moved R10 57.0 mm to (56.7, 82.5), turned to -90 degrees
- moved R12 56.5 mm to (56.4, 72.4), turned to -90 degrees
- moved C43 56.3 mm to (118.8, 82.3), turned to -90 degrees
- moved R13 56.0 mm to (56.7, 77.0), turned to -90 degrees
- moved SW5 52.5 mm to (63.8, 92.8), turned to 180 degrees
- moved SW4 49.4 mm to (63.8, 87.6), turned to 180 degrees
- moved SW3 47.2 mm to (63.8, 82.5), turned to 180 degrees
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Connections:
- net /D+ renamed /MCU/D+
- net /D- renamed /MCU/D-
- net /Ft232/FT_DRS renamed /Ft232/FT_DSR
- net /MCU/RB12 renamed /AN12
- net /MCU/RB13 renamed /AN14
- net /MCU/RB14 renamed /AN13
- net Net-(A1-1A) renamed /Pololu/1A_1
- net Net-(A1-1B) renamed /Pololu/1B_1
- net Net-(A1-2A) renamed /Pololu/2A_1
- net Net-(A1-2B) renamed /Pololu/2B_1
- net Net-(A1-MS1) renamed /Pololu/MS1_DRV8825_1
- net Net-(A1-MS2) renamed /Pololu/MS2_DRV8825_1
- net Net-(A1-MS3) renamed /Pololu/MS3_DRV8825_1
- net Net-(A2-1A) renamed /Pololu/1A_2
- net Net-(A2-1B) renamed /Pololu/1B_2
- net Net-(A2-2A) renamed /Pololu/2A_2
- net Net-(A2-2B) renamed /Pololu/2B_2
- net Net-(A2-MS1) renamed /Pololu/MS1_DRV8825_2
- net Net-(A2-MS2) renamed /Pololu/MS2_DRV8825_2
- net Net-(A2-MS3) renamed /Pololu/MS3_DRV8825_2
- net Net-(A3-1A) renamed /Pololu/1A_3
- net Net-(A3-1B) renamed /Pololu/1B_3
- net Net-(A3-2A) renamed /Pololu/2A_3
- net Net-(A3-2B) renamed /Pololu/2B_3
- net Net-(A3-MS1) renamed /Pololu/MS1_DRV8825_3
- net Net-(A3-MS2) renamed /Pololu/MS2_DRV8825_3
- net Net-(A3-MS3) renamed /Pololu/MS3_DRV8825_3
- net Net-(A4-1A) renamed /Pololu/1A_4
- net Net-(A4-1B) renamed /Pololu/1B_4
- net Net-(A4-2A) renamed /Pololu/2A_4
- net Net-(A4-2B) renamed /Pololu/2B_4
- net Net-(A4-MS1) renamed /Pololu/MS1_DRV8825_4
- net Net-(A4-MS2) renamed /Pololu/MS2_DRV8825_4
- net Net-(A4-MS3) renamed /Pololu/MS3_DRV8825_4
- net Net-(A5-1A) renamed /Pololu/1A_5
- net Net-(A5-1B) renamed /Pololu/1B_5
- net Net-(A5-2A) renamed /Pololu/2A_5
- net Net-(A5-2B) renamed /Pololu/2B_5
- net Net-(A5-MS1) renamed /Pololu/MS1_DRV8825_5
- net Net-(A5-MS2) renamed /Pololu/MS2_DRV8825_5
- net Net-(A5-MS3) renamed /Pololu/MS3_DRV8825_5
- A1 pad 13: /MCU/RA0 -> /MCU/RA1
- A1 pad 14: /MCU/RA1 -> /MCU/RB15
- A1 pad 15: /MCU/RA3 -> /MCU/RB10
- A1 pad 16: /MCU/RA4 -> /MCU/RB11
- A1 pad 2: +5V -> +3.3V
- A1 pad 8: +3.3V -> VCC
- A1 pad 9: /MCU/RA2 -> /MCU/RB9
- A2 pad 13: /MCU/RA5 -> /MCU/RA1
- A2 pad 14: /MCU/RA6 -> /MCU/RB15
- A2 pad 15: /MCU/RA9 -> /MCU/RA10
- A2 pad 16: /MCU/RA10 -> /MCU/RB2
- A2 pad 2: +5V -> +3.3V
- A2 pad 8: +3.3V -> VCC
- A2 pad 9: /MCU/RA7 -> /MCU/RA9
- A3 pad 13: /MCU/PGC1 -> /MCU/RA1
- A3 pad 14: /MCU/PGD1 -> /MCU/RB15
- A3 pad 15: /MCU/RB3 -> /MCU/RE8
- A3 pad 16: /MCU/PGM -> /MCU/RE9
- A3 pad 2: +5V -> +3.3V
- A3 pad 8: +3.3V -> VCC
- A3 pad 9: /MCU/RB2 -> /MCU/RB5
- A4 pad 13: /MCU/RE9 -> /MCU/RA1
- A4 pad 14: /MCU/RE8 -> /MCU/RB15
- A4 pad 15: /MCU/RE6 -> /MCU/RC3
- A4 pad 16: /MCU/RE5 -> /MCU/RG6
- A4 pad 2: +5V -> +3.3V
- A4 pad 8: +3.3V -> VCC
- A4 pad 9: /MCU/RE7 -> /MCU/RC2
- A5 pad 13: /MCU/RE4 -> /MCU/RA1
- A5 pad 14: /MCU/RE3 -> /MCU/RB15
- A5 pad 15: /MCU/RE1 -> /MCU/RE7
- A5 pad 16: /MCU/RE0 -> /MCU/RE6
- A5 pad 2: +5V -> +3.3V
- A5 pad 8: +3.3V -> VCC
- A5 pad 9: /MCU/RE2 -> /MCU/RC1
- C14 pad 2: +5V -> Net-(U2-VI)
- C29 pad 1: +5V -> VCC
- C31 pad 1: +5V -> VCC
- C32 pad 1: +5V -> VCC
- C33 pad 1: +5V -> VCC
- C34 pad 1: +5V -> VCC
- C35 pad 1: +5V -> VCC
- C36 pad 1: +5V -> VCC
- C38 pad 2: +5V -> Net-(U2-VI)
- C39 pad 1: +5V -> VCC
- C40 pad 1: +5V -> VCC
- C41 pad 1: +5V -> VCC
- C45 pad 1: +12V -> +3.3V
- C47 pad 1: +12V -> +3.3V
- C48 pad 1: +5V -> VCC
- C49 pad 1: +5V -> VCC
- C50 pad 1: +5V -> VCC
- J2 pad 1: Net-(J2-VBUS) -> /MCU/VBUS
- J2 pad 4: unconnected-(J2-ID-Pad4) -> /MCU/RF3
- J21 pad 2: +5V -> unconnected-(J21-Pin_2-Pad2)
- J21 pad 3: /MCU/RA15 -> /Oled/sda_i2c_2
- J21 pad 4: +5V -> unconnected-(J21-Pin_4-Pad4)
- J21 pad 5: /MCU/RA14 -> /Oled/scl_i2c_2
- J25 pad 3: /MCU/RG6 -> /MCU/RA2
- J25 pad 4: /MCU/RG8 -> /MCU/RA3
- L1 pad 1: Net-(J2-VBUS) -> /MCU/VBUS
- L1 pad 2: +5V -> Net-(U2-VI)
- R10 pad 2: /RD5 -> /MCU/RD9
- R11 pad 2: /RD4 -> /MCU/RD8
- R12 pad 1: +12V -> VCC
- R14 pad 2: /RD7 -> /MCU/RD12
- R15 pad 2: /RD6 -> /MCU/RD11
- R3 pad 1: /Ft232/TX -> Net-(D6-K)
- R3 pad 2: +5VA -> GND
- R33 pad 2: /MCU/RF4 -> /MCU/RD2
- R34 pad 2: /MCU/RF12 -> /MCU/RF0
- R37 pad 1: /MCU/RF3 -> /MCU/RD14
- R38 pad 2: /MCU/RF1 -> /MCU/RD15
- R39 pad 2: /MCU/RF0 -> /MCU/RF8
- SW2 pad 1: /RD4 -> /MCU/RD8
- SW3 pad 1: /RD5 -> /MCU/RD9
- SW4 pad 1: /RD6 -> /MCU/RD11
- SW5 pad 1: /RD7 -> /MCU/RD12
- U1 pad 11: /MCU/RG7 -> /U4RX
- U1 pad 12: /MCU/RG8 -> /U4TX
- U1 pad 47: /U4RX -> /MCU/RD14
- U1 pad 48: /U4TX -> /MCU/RD15
- U1 pad 72: /M1 -> /MCU/RD0
- U1 pad 81: /RD4 -> /MCU/RD4
- U1 pad 82: /RD5 -> /MCU/RD5
- U1 pad 83: /RD6 -> /MCU/RD6
- U1 pad 84: /RD7 -> /MCU/RD7
- U1 pad 89: /MCU/RG1 -> /M1
- U2 pad 3: +5V -> Net-(U2-VI)
- U7 pad 11: /MCU/RG7 -> /U4RX
- U7 pad 12: /MCU/RG8 -> /U4TX
- U7 pad 47: /U4RX -> /MCU/RD14
- U7 pad 48: /U4TX -> /MCU/RD15
- U7 pad 81: /RD4 -> /MCU/RD4
- U7 pad 82: /RD5 -> /MCU/RD5
- U7 pad 83: /RD6 -> /MCU/RD6
- U7 pad 84: /RD7 -> /MCU/RD7
- U7 pad 89: /MCU/RG1 -> /M1
- U8 pad 1: /MCU/RF4 -> /MCU/RD2
- U8 pad 13: /MCU/RF0 -> /MCU/RF8
- U8 pad 14: /MCU/RF1 -> /MCU/RD15
- U8 pad 3: /MCU/RF5 -> /MCU/RF1
- U8 pad 9: /MCU/RF3 -> /MCU/RD14
Routing:
- added copper zone on B.Cu, net GND
- added copper zone on F.Cu, net GND

Commit message: LPCXpresso
Parts:
- removed C11: 100nf, Capacitor_SMD:C_0805_2012Metric
- removed J1: icd, Connector_PinHeader_2.54mm:PinHeader_1x06_P2.54mm_Vertical
- removed U1: PIC32MX795F512L-80x-PF, Package_QFP:TQFP-100_14x14mm_P0.5mm
- removed U7: PIC32MX795F512L-80x-PF, altium:MA240011_Socket_TQFP100_100pin
- added LPC1: LPCXPRESSO_LPC1769, Libraries:LPCXPRESSO_LPC1769, F.Cu at (89.5, -3.68)
- added U5: LPC1769FBD100, Package_QFP:LQFP-100_14x14mm_P0.5mm, F.Cu at (95.4, 74.8)
- J24: value Micro_SD_Card -> TF-001B
- U8: moved to B.Cu
- moved J21 40.6 mm to (53.9, 51.7)
- moved R38 39.7 mm to (88.9, 52.2)
- moved R39 39.1 mm to (99.8, 55.0)
- moved C4 35.7 mm to (100.1, 57.2)
- moved C13 30.7 mm to (91.9, 57.5), turned to 0 degrees
- moved R6 29.8 mm to (96.3, 54.4), turned to 0 degrees
- moved R7 26.3 mm to (96.3, 57.4), turned to 0 degrees
- moved C28 25.0 mm to (102.4, 52.0)
- moved R1 25.0 mm to (103.2, 55.5)
- moved C15 25.0 mm to (93.9, 57.3)
- moved C12 24.2 mm to (91.9, 54.5)
- moved Y1 23.2 mm to (93.7, 61.5), turned to 0 degrees
- moved D8 23.0 mm to (98.7, 33.1), turned to 90 degrees
- moved R41 22.7 mm to (116.7, 32.2)
- moved D3 22.7 mm to (118.9, 28.2)
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Connections:
- C13 pad 1: /MCU/MA240011/OSC1 -> /MCU/OSC1
- R6 pad 1: /MCU/MA240011/OSC2 -> /MCU/OSC2
- R7 pad 2: /MCU/MA240011/OSC1 -> /MCU/OSC1
- Y1 pad 3: /MCU/MA240011/OSC1 -> /MCU/OSC1
