File: mcu.kicad_sch (KiCad schematic)
At the start: 3 parts, among them U1 PIC32MX795F512L-80x-PF

Commit message: LPCXpresso
Parts:
- added C12, C13: 15p, Capacitor_SMD:C_0805_2012Metric, symbol Device:C
- added LPC1: LPCXPRESSO_LPC1769, Libraries:LPCXPRESSO_LPC1769, symbol LPCXPRESSO_LPC1769:LPCXPRESSO_LPC1769
- added R6: 1K, Resistor_SMD:R_0805_2012Metric, symbol Device:R
- added R7: 1M, Resistor_SMD:R_0805_2012Metric, symbol Device:R
- added U5: LPC1769FBD100, Package_QFP:LQFP-100_14x14mm_P0.5mm, symbol MCU_NXP_LPC:LPC1769FBD100
- added Y1: 8MHz SMD crystal oscillator ±10ppm ±30ppm SMD3225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, Crystal:Crystal_SMD_3225-4Pin_3.2x2.5mm, symbol Device:Crystal_GND24
- U1: now not fitted; now left out of the parts list
Connections:
- net +3.3V: now also LPC1.28, U5.10 (VDDA), U5.12 (VREFP), U5.19 (VBAT), U5.28 (VDD(3V3)), U5.42 (VDD(REG)(3V3)), U5.54 (VDD(3V3)), U5.71 (VDD(3V3)), U5.84 (VDD(REG)(3V3)), U5.96 (VDD(3V3))
- net D+: now also LPC1.37
- net D-: now also LPC1.36
- net GND: now also C12.2, C13.2, LPC1.1, LPC1.54, U5.11 (VSSA), U5.15 (VREFN), U5.31 (VSS), U5.41 (VSS), U5.55 (VSS), U5.72 (VSS), U5.83 (VSS), U5.97 (VSS), Y1.2, Y1.4
- net OSC1: now also C13.1, R7.2, U5.22 (XTAL1), Y1.3; no longer U1.63 (RC12/OSC1/CLK)
- net OSC2: now also R6.1, U5.23 (XTAL2); no longer U1.64 (RC15/OSC2/CLKO)
- net RA0: now also LPC1.38
- net RA1: now also LPC1.70, U5.35 (P1[21])
- net RA10: now also LPC1.52, U5.52 (P2[11])
- net RA9: now also LPC1.53, U5.51 (P2[12])
- net RB10: now also LPC1.73, U5.32 (P1[18])
- net RB11: now also LPC1.68, U5.37 (P1[23])
- net RB15: now also LPC1.69, U5.36 (P1[22])
- net RB2: now also LPC1.51, U5.53 (P2[10])
- net RB3: now also LPC1.50, U5.65 (P2[8])
- net RB5: now also LPC1.49, U5.66 (P2[7])
- net RB8: now also LPC1.71, U5.34 (P1[20])
- net RB9: now also LPC1.72, U5.33 (P1[19])
- net RC1: now also LPC1.42, U5.75 (P2[0])
- net RC2: now also LPC1.41
- net RC3: now also LPC1.40, U5.48 (P0[10])
- net RE5: now also LPC1.45, U5.70 (P2[3])
- net RE6: now also LPC1.44, U5.73 (P2[2])
- net RE7: now also LPC1.43, U5.74 (P2[1])
- net RE8: now also LPC1.48, U5.67 (P2[6])
- net RE9: now also LPC1.47, U5.68 (P2[5])
- net RG6: now also LPC1.39
- net RG9: now also LPC1.46, U5.69 (P2[4])
- new net: C12.1, R6.2, R7.1, Y1.1
- new net RESET: U5.17 (~{RESET})
- new net RSTOUT: U5.14 (~{RSTOUT})
- new net RTCK: U5.100 (RTCK)
- new net RTCX1: U5.16 (RTCX1)
- new net RTCX2: U5.18 (RTCX2)
- new net TCK: U5.5 (TCK/SWDCLK)
- new net TDI: U5.2 (TDI)
- new net TDO: U5.1 (TDO/SWO)
- new net TMS: U5.3 (TMS/SWDIO)
- new net TRST: U5.4 (~{TRST})
- new net p0_0: LPC1.9, U5.46 (P0[0])
- new net p0_1: LPC1.10, U5.47 (P0[1])
- new net p0_11: U5.49 (P0[11])
- new net p0_15: LPC1.13, U5.62 (P0[15])
- new net p0_16: LPC1.14, U5.63 (P0[16])
- new net p0_17: LPC1.12, U5.61 (P0[17])
- new net p0_18: LPC1.11, U5.60 (P0[18])
- new net p0_19: LPC1.57, U5.59 (P0[19])
- new net p0_2: LPC1.21, U5.98 (P0[2])
- new net p0_20: LPC1.56, U5.58 (P0[20])
- new net p0_21: LPC1.23, U5.57 (P0[21])
- new net p0_22: LPC1.24, U5.56 (P0[22])
- new net p0_23: LPC1.15, U5.9 (P0[23])
- new net p0_24: LPC1.16, U5.8 (P0[24])
- new net p0_25: LPC1.17, U5.7 (P0[25])
- new net p0_26: LPC1.18, U5.6 (P0[26])
- new net p0_27: LPC1.25, U5.25 (P0[27])
- new net p0_28: LPC1.26, U5.24 (P0[28])
- new net p0_29: U5.29 (P0[29])
- new net p0_3: LPC1.22, U5.99 (P0[3])
- new net p0_30: U5.30 (P0[30])
- new net p0_4: U5.81 (P0[4])
- new net p0_5: U5.80 (P0[5])
- new net p0_6: LPC1.8, U5.79 (P0[6])
- new net p0_7: LPC1.7, U5.78 (P0[7])
- new net p0_8: LPC1.6, U5.77 (P0[8])
- new net p0_9: LPC1.5, U5.76 (P0[9])
- new net p1_0: U5.95 (P1[0])
- new net p1_1: U5.94 (P1[1])
- new net p1_10: U5.90 (P1[10])
- new net p1_14: U5.89 (P1[14])
- new net p1_15: U5.88 (P1[15])
- new net p1_16: U5.87 (P1[16])
- new net p1_17: U5.86 (P1[17])
- new net p1_24: LPC1.67, U5.38 (P1[24])
- new net p1_25: LPC1.66, U5.39 (P1[25])
- new net p1_26: LPC1.65, U5.40 (P1[26])
- new net p1_27: LPC1.62, U5.43 (P1[27])
- new net p1_28: LPC1.63, U5.44 (P1[28])
- new net p1_29: LPC1.64, U5.45 (P1[29])
- new net p1_30: LPC1.19, U5.21 (P1[30])
- new net p1_31: LPC1.20, U5.20 (P1[31])
- new net p1_4: U5.93 (P1[4])
- new net p1_8: U5.92 (P1[8])
- new net p1_9: U5.91 (P1[9])
- new net p2_13: LPC1.27, U5.50 (P2[13])
- new net p2_9: LPC1.55, U5.64 (P2[9])
- new net p3_25: LPC1.61, U5.27 (P3[25])
- new net p3_26: LPC1.60, U5.26 (P3[26])
- new net p4_28: LPC1.59, U5.82 (P4[28])
- new net p4_29: LPC1.58, U5.85 (P4[29])
Other:
- moved on the sheet: R1, R43
