File: mcu.kicad_sch (KiCad schematic)
At the start: 6 parts, among them U1 PIC32MX795F512L-80x-PF

Commit message: CNC Raspberry update
Parts:
- removed R10, R13: 10K, Resistor_SMD:R_0805_2012Metric, symbol Device:R
- removed R11, R12: 0, Resistor_SMD:R_0805_2012Metric, symbol Device:R
- removed R14: 100, Resistor_SMD:R_0805_2012Metric, symbol Device:R
- removed U1: PIC32MX795F512L-80x-PF, Package_QFP:TQFP-100_14x14mm_P0.5mm, symbol MCU_Microchip_PIC32:PIC32MX795F512L-80x-PF
- added J1, J9: Raspberry_Pi_4, Connector_PinHeader_2.54mm:PinHeader_2x20_P2.54mm_Vertical, symbol Connector:Raspberry_Pi_4
Connections:
- net +3.3V: now also J1.1 (3V3), J1.17 (3V3), J9.1 (3V3), J9.17 (3V3)
- net GND: now also J1.14 (GND), J1.20 (GND), J1.25 (GND), J1.30 (GND), J1.34 (GND), J1.39 (GND), J1.6 (GND), J1.9 (GND), J9.14 (GND), J9.20 (GND), J9.25 (GND), J9.30 (GND), J9.34 (GND), J9.39 (GND), J9.6 (GND), J9.9 (GND)
- new net +5V: J1.2 (5V), J1.4 (5V), J9.2 (5V), J9.4 (5V)
- new net CE0: J1.24 (~{CE0}_SPI0/GPIO08), J9.24 (~{CE0}_SPI0/GPIO08)
- new net CE1: J1.26 (~{CE1}_SPI0/GPIO07), J9.26 (~{CE1}_SPI0/GPIO07)
- new net GPIO2_SDA: J1.3 (SDA_I2C1/GPIO02), J9.3 (SDA_I2C1/GPIO02)
- new net GPIO3_SCL: J1.5 (SCL_I2C1/GPIO03), J9.5 (SCL_I2C1/GPIO03)
- new net GPIO_0: J1.27 (ID_SD_I2C0/GPIO00), J9.27 (ID_SD_I2C0/GPIO00)
- new net GPIO_1: J1.28 (ID_SC_I2C0/GPIO01), J9.28 (ID_SC_I2C0/GPIO01)
- new net GPIO_16: J1.36 (GPIO16/SPI1_~{CE2}), J9.36 (GPIO16/SPI1_~{CE2})
- new net GPIO_17: J1.11 (GPIO17/SPI1_~{CE1}), J9.11 (GPIO17/SPI1_~{CE1})
- new net GPIO_18: J1.12 (GPIO18/SPI1_~{CE0}/PCM_CLK/PWM0), J9.12 (GPIO18/SPI1_~{CE0}/PCM_CLK/PWM0)
- new net GPIO_19: J1.35 (GPIO19/SPI1_MISO/PCM_FS), J9.35 (GPIO19/SPI1_MISO/PCM_FS)
- new net GPIO_20: J1.38 (GPIO20/SPI1_MOSI/PCM_DIN/PWM1), J9.38 (GPIO20/SPI1_MOSI/PCM_DIN/PWM1)
- new net GPIO_21: J1.40 (GPIO21/SPI1_SCLK/PCM_DOUT), J9.40 (GPIO21/SPI1_SCLK/PCM_DOUT)
- new net GPIO_22: J1.15 (GPIO22/SDIO_CLK), J9.15 (GPIO22/SDIO_CLK)
- new net GPIO_23: J1.16 (GPIO23/SDIO_CMD), J9.16 (GPIO23/SDIO_CMD)
- new net GPIO_24: J1.18 (GPIO24/SDIO_DAT0), J9.18 (GPIO24/SDIO_DAT0)
- new net GPIO_25: J1.22 (GPIO25/SDIO_DAT1), J9.22 (GPIO25/SDIO_DAT1)
- new net GPIO_26: J1.37 (GPIO26/SDIO_DAT2), J9.37 (GPIO26/SDIO_DAT2)
- new net GPIO_27: J1.13 (GPIO27/SDIO_DAT3), J9.13 (GPIO27/SDIO_DAT3)
- new net GPIO_4: J1.7 (GPCLK0/GPIO04), J9.7 (GPCLK0/GPIO04)
- new net GPIO_5: J1.29 (GPCLK1/GPIO05), J9.29 (GPCLK1/GPIO05)
- new net GPIO_6: J1.31 (GPCLK2/GPIO06), J9.31 (GPCLK2/GPIO06)
- new net MISO: J1.21 (MISO_SPI0/GPIO09), J9.21 (MISO_SPI0/GPIO09)
- new net MOSI: J1.19 (MOSI_SPI0/GPIO10), J9.19 (MOSI_SPI0/GPIO10)
- new net MRX: J1.10 (GPIO15/UART_RXD), J9.10 (GPIO15/UART_RXD)
- new net MTX: J1.8 (GPIO14/UART_TXD), J9.8 (GPIO14/UART_TXD)
- new net PWM0: J1.32 (GPIO12/PWM0), J9.32 (GPIO12/PWM0)
- new net PWM1: J1.33 (GPIO13/PWM1), J9.33 (GPIO13/PWM1)
- new net SCLK: J1.23 (SCLK_SPI0/GPIO11), J9.23 (SCLK_SPI0/GPIO11)
- no-connect marks 0 -> 1
Other:
- removed sheet buttons

Commit message: update sch & pcb
Parts:
- removed J9: Raspberry_Pi_4, Connector_PinHeader_2.54mm:PinHeader_2x20_P2.54mm_Vertical, symbol Connector:Raspberry_Pi_4
- added U10: 74HC595, kiC:SOIC-16_3.9x9.9mm_P1.27mm, symbol 74xx:74HC595
- J1: footprint Connector_PinHeader_2.54mm:PinHeader_2x20_P2.54mm_Vertical -> kiC:Rpi_PinHeader_2x20_P2.54mm_Vertical
Connections:
- net +3.3V: now also U10.10 (~{SRCLR}), U10.16 (VCC)
- net GND: now also U10.13 (~{OE}), U10.8 (GND)
- new net QA: U10.15 (QA)
- new net QB: U10.1 (QB)
- new net QC: U10.2 (QC)
- new net QD: U10.3 (QD)
- new net QE: U10.4 (QE)
- new net QF: U10.5 (QF)
- new net QG: U10.6 (QG)
- new net QH: U10.7 (QH)
- new net gpio22: U10.14 (SER)
- new net gpio24: U10.12 (RCLK)
- new net gpio_23: U10.11 (SRCLK)
- no-connect marks 1 -> 2
