File: buttons.kicad_sch (KiCad schematic)
At the start: 11 parts, among them SW1 power, SW2 up, SW3 down, SW4 left, SW5 rigth

Commit message: Clear remaining KiCad 10-only footprints: SW_Push, kiC, MODULE_MRF24J40MA
Parts:
- SW1, SW3, SW4, SW5: footprint Button_Switch_SMD:SW_Push_1P1T_NO_6x6mm_H9.5mm -> (none)
Changed lines of the file:
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@@
 			)
 		)
-		(property "Footprint" "Button_Switch_SMD:SW_Push_1P1T_NO_6x6mm_H9.5mm"
+		(property "Footprint" ""
 			(at 212.09 110.49 0)
 			(hide yes)
@@
 			)
 		)
-		(property "Footprint" "Button_Switch_SMD:SW_Push_1P1T_NO_6x6mm_H9.5mm"
+		(property "Footprint" ""
 			(at 137.16 77.47 0)
 			(hide yes)
@@
 			)
 		)
-		(property "Footprint" "Button_Switch_SMD:SW_Push_1P1T_NO_6x6mm_H9.5mm"
+		(property "Footprint" ""
 			(at 144.78 123.19 0)
 			(hide yes)
@@
 			)
 		)
-		(property "Footprint" "Button_Switch_SMD:SW_Push_1P1T_NO_6x6mm_H9.5mm"
+		(property "Footprint" ""
 			(at 212.09 97.79 0)
 			(hide yes)

Commit message: Extraer footprints de example.kicad_pcb y asignarlos a los esquematicos
Parts:
- SW1, SW3, SW4, SW5: footprint (none) -> custom:SW_Push_1P1T_NO_6x6mm_H9.5mm
Changed lines of the file:
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@@
 			)
 		)
-		(property "Footprint" ""
+		(property "Footprint" "custom:SW_Push_1P1T_NO_6x6mm_H9.5mm"
 			(at 212.09 110.49 0)
 			(hide yes)
@@
 			)
 		)
-		(property "Footprint" ""
+		(property "Footprint" "custom:SW_Push_1P1T_NO_6x6mm_H9.5mm"
 			(at 137.16 77.47 0)
 			(hide yes)
@@
 			)
 		)
-		(property "Footprint" ""
+		(property "Footprint" "custom:SW_Push_1P1T_NO_6x6mm_H9.5mm"
 			(at 144.78 123.19 0)
 			(hide yes)
@@
 			)
 		)
-		(property "Footprint" ""
+		(property "Footprint" "custom:SW_Push_1P1T_NO_6x6mm_H9.5mm"
 			(at 212.09 97.79 0)
 			(hide yes)

Commit message: CNC Raspberry update
Parts:
- added D6, D7, D8: LED, Diode_SMD:D_0805_2012Metric, symbol Device:LED
- added R3, R50, R51: 1k, Resistor_SMD:R_0805_2012Metric, symbol Device:R
- R14: renamed from R62; footprint Resistor_SMD:R_0603_1608Metric -> Resistor_SMD:R_0805_2012Metric
- R15: renamed from R63; footprint Resistor_SMD:R_0603_1608Metric -> Resistor_SMD:R_0805_2012Metric
- SW1: value power -> K2-1107ST-A4SW-06; footprint custom:SW_Push_1P1T_NO_6x6mm_H9.5mm -> Button_Switch_SMD:SW_Tactile_SPST_NO_Straight_CK_PTS636Sx25SMTRLFS
- SW2: value up -> K2-1107ST-A4SW-06; footprint Button_Switch_SMD:SW_SPST_CK_RS282G05A3 -> Button_Switch_SMD:SW_Tactile_SPST_NO_Straight_CK_PTS636Sx25SMTRLFS
- SW3: value down -> K2-1107ST-A4SW-06; footprint custom:SW_Push_1P1T_NO_6x6mm_H9.5mm -> Button_Switch_SMD:SW_Tactile_SPST_NO_Straight_CK_PTS636Sx25SMTRLFS
- SW4: value left -> K2-1107ST-A4SW-06; footprint custom:SW_Push_1P1T_NO_6x6mm_H9.5mm -> Button_Switch_SMD:SW_Tactile_SPST_NO_Straight_CK_PTS636Sx25SMTRLFS
- SW5: value rigth -> K2-1107ST-A4SW-06; footprint custom:SW_Push_1P1T_NO_6x6mm_H9.5mm -> Button_Switch_SMD:SW_Tactile_SPST_NO_Straight_CK_PTS636Sx25SMTRLFS
- renumbered R57 to R10, R58 to R11, R59 to R12, R60 to R13
Connections:
- net GND: now also R3.2, R50.2, R51.2
- net SW5: now reaches R14.2, SW5.1
- net SW4: now reaches R15.2, SW4.1
- net SW3: now reaches R10.2, SW3.1
- net SW2: now reaches R11.2, SW2.1
- net +12V renamed VCC
- new net: D8.1 (K), R51.1
- new net: D7.1 (K), R50.1
- new net: D6.1 (K), R3.1
- new net led1: D6.2 (A)
- new net led2: D7.2 (A)
- new net led3: D8.2 (A)
Other:
- note added: "posible push C49234124 otro recomendado C118141 4 patas comprado en mouser C127478 switch value SKQGAKE010 4 patas C127478 foot: Button_Switch_SMD:SW_SPST_TL3342"
