File: cnc_pic32.kicad_sch (KiCad schematic)
At the start: 0 parts

Commit message: CNC Raspberry update
Connections:
- no-connect marks 0 -> 21
Other:
- removed sheet Usb_pic32
- removed sheet idc
- removed sheet oscilator
- removed sheet zigbee
- added sheet Radio (zigbee.kicad_sch)
- added sheet buttons (buttons.kicad_sch)
- added sheet microSD (microSD.kicad_sch)
- sheet Ft232 ports: added FT_CTS, FT_DTR, FT_RX, FT_TX, FT_VCC, MCLR; removed RX_MCU, TX_MCU, mclr
- sheet MCU ports: added CE0, CE1, GPIO2_SDA, GPIO3_SCL, GPIO_0, GPIO_1, GPIO_16, GPIO_17, GPIO_18, GPIO_19, GPIO_20, GPIO_21, GPIO_22, GPIO_23, GPIO_24, GPIO_25, GPIO_26, GPIO_27, GPIO_4, GPIO_5, GPIO_6, MISO, MOSI, MRX, MTX, PWM0, PWM1, SCLK; removed D+, D-, OSC1, OSC2, RA0, RA1, RA10, RA14, RA15, RA2, RA3, RA4, RA5, RA6, RA7, RA9, RB0, RB1, RB10, RB11, RB12, RB13, RB14, RB15, RB2, RB3, RB4, RB5, RB6, RB7, RB8, RB9, RC1, RC2, RC3, RC4, RD0, RD1, RD10, RD11, RD12, RD13, RD14, RD15, RD2, RD3, RD4, RD5, RD6, RD7, RD8, RD9, RE0, RE1, RE2, RE3, RE4, RE5, RE6, RE7, RE8, RE9, RF0, RF1, RF12, RF13, RF2, RF3, RF4, RF5, RF8, RG0, RG1, RG12, RG13, RG14, RG15, RG6, RG7, RG8, RG9, SOSC0, SOSC1, VBUS, mclr
- sheet Oled ports: added scl_i2c_1, sda_i2c_1; removed none
- sheet Pololu ports: added FLT_1, FLT_2, FLT_3, FLT_4, FLT_5, MS1, MS2, MS3, dir_1, dir_2, dir_3, dir_4, dir_5, enable_1, enable_2, enable_3, enable_4, enable_5, reset, sleep, step_1, step_2, step_3, step_4, step_5; removed none
