File: idc.kicad_sch (KiCad schematic)
At the start: 2 parts, among them J1 icd

Commit message: CNC Raspberry update
Parts:
- removed C8: 100nf, Capacitor_SMD:C_0805_2012Metric, symbol Device:C
- removed J1: icd, Connector_PinHeader_2.54mm:PinHeader_1x06_P2.54mm_Horizontal, symbol Connector:Conn_01x06_Pin
