File: oled.kicad_sch (KiCad schematic)
At the start: 4 parts, among them J2 ST7789 oled 128x64, J23 conector oled ST1306 128x32

Commit message: Clear remaining KiCad 10-only footprints: SW_Push, kiC, MODULE_MRF24J40MA
Parts:
- J2: footprint kiC:Adafruit_SSD1306_No_Mounting_Holes_pads -> (none)
Changed lines of the file:
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@@
 			)
 		)
-		(property "Footprint" "kiC:Adafruit_SSD1306_No_Mounting_Holes_pads"
+		(property "Footprint" ""
 			(at 189.23 82.55 0)
 			(hide yes)

Commit message: Extraer footprints de example.kicad_pcb y asignarlos a los esquematicos
Parts:
- J2: footprint (none) -> custom:Adafruit_SSD1306_No_Mounting_Holes_pads
Changed lines of the file:
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@@
 			)
 		)
-		(property "Footprint" ""
+		(property "Footprint" "custom:Adafruit_SSD1306_No_Mounting_Holes_pads"
 			(at 189.23 82.55 0)
 			(hide yes)

Commit message: CNC Raspberry update
Parts:
- removed J2: ST7789 oled 128x64, custom:Adafruit_SSD1306_No_Mounting_Holes_pads, symbol Connector:Conn_01x07_Pin
- added J23: OLED SSD1306, Connector_PinHeader_2.54mm:PinHeader_1x04_P2.54mm_Vertical, symbol Connector:Conn_01x04_Pin
- J21: renamed from J23; now left out of the parts list
- renumbered R42 to R31, R41 to R32
Connections:
- net +3.3V: now also J21.1 (Pin_1), J23.2 (Pin_2); no longer J21.2 (Pin_2)
- net GND: now also J21.6 (Pin_6), J23.1 (Pin_1); no longer J21.1 (Pin_1)
- net scl_i2c_1: now reaches J21.5 (Pin_5)
- net scl_i2c_1: now also R31.2, J23.3 (Pin_3)
- net scl renamed sda_i2c_1
- net sda_i2c_1: now also R32.2, J23.4 (Pin_4); no longer R31.2
- net sda: no longer names the net of J21.4 (Pin_4)
- net sda: no longer R32.2
- no-connect marks 0 -> 2
Other:
- moved on the sheet: R31
