File: oscilator.kicad_sch (KiCad schematic)
At the start: 5 parts, among them Y1 8Mhz

Commit message: CNC Raspberry update
Parts:
- removed Y1: 8Mhz, symbol Device:Crystal
- added Y1: 8MHZ, Crystal:Crystal_SMD_0603-4Pin_6.0x3.5mm, symbol Device:Crystal_GND24
- renumbered C9 to C12, C10 to C13, R15 to R6, R16 to R7
Connections:
- net GND: now also Y1.2, Y1.4
- net OSC1: now also Y1.3
- net at C12.1, R6.2, R7.1: now also Y1.1
- net OSC0 renamed OSC2
Other:
- moved on the sheet: R6
