File: power.kicad_sch (KiCad schematic)
At the start: 10 parts

Commit message: CNC Raspberry update
Parts:
- removed C26, C27, C28: 100nf, Capacitor_SMD:C_0805_2012Metric, symbol Device:C
- added C14, C15, C36: 4.7uf, Capacitor_SMD:C_0805_2012Metric, symbol Device:C
- added C29, C31, C32, C33, C34, C35, C57, C58, C59, C60: 100nf, Capacitor_SMD:C_0805_2012Metric, symbol Device:C
- added C38: 100nf, Capacitor_SMD:C_1206_3216Metric, symbol Device:C
- added C39, C40, C41, C48, C49, C50: RVT100UF35V67RV0034, Capacitor_SMD:C_Elec_6.3x5.4, symbol Device:C_Polarized
- added C42, C43, C45, C47, C51, C52: EFVH035ADA100M0454, Capacitor_SMD:C_Elec_5x5.4, symbol Device:C_Polarized
- added J2: USB_B_Mini, Library:USB_Mini-B_Wuerth_65100516121_Horizontal, symbol Connector:USB_B_Mini
- added L1: 100mh, Inductor_SMD:L_1210_3225Metric, symbol Device:L
- added R42: 0, Resistor_SMD:R_0805_2012Metric, symbol Device:R
- added R8, R9: 22, Resistor_SMD:R_0805_2012Metric, symbol Device:R
- added U2: LM1117DT-3.3, Package_TO_SOT_SMD:TO-252-3_TabPin2, symbol Regulator_Linear:LM1117DT-3.3
- C3, C4: footprint Capacitor_SMD:C_0805_2012Metric -> Resistor_SMD:R_0603_1608Metric
- renumbered C24 to C6, C25 to C7
Connections:
- net +3.3V: now also C42.1, C43.1, C45.1, C47.1, C51.1, C52.1
- net GND: now also C14.1, C15.1, C29.2, C31.2, C32.2, C33.2, C34.2, C35.2, C36.2, C38.1, C39.2, C40.2, C41.2, C42.2, C43.2, C45.2, C47.2, C48.2, C49.2, C50.2, C51.2, C52.2, C57.2, C58.2, C59.2, C60.2, R42.1, U2.1 (GND)
- new net: J2.1 (VBUS), L1.1
- new net: C14.2, C38.2, L1.2, U2.3 (VI)
- new net: J2.5 (GND), R42.2
- new net +3V3: C15.2, U2.2 (VO)
- new net D+: R8.1
- new net D-: R9.1
- new net USB_D+: J2.3 (D+), R8.2
- new net USB_D-: J2.2 (D-), R9.2
- new net VCC: C29.1, C31.1, C32.1, C33.1, C34.1, C35.1, C36.1, C39.1, C40.1, C41.1, C48.1, C49.1, C50.1, C57.1, C58.1, C59.1, C60.1
- no-connect marks 0 -> 4
