File: power_ft232.kicad_sch (KiCad schematic)
At the start: 5 parts

Commit message: CNC Raspberry update
Parts:
- renumbered C18 to C23, C19 to C24, C20 to C25, C21 to C26, R31 to R30
Other:
- moved on the sheet: C25, C26, R30
